File: tp_ft232.kicad_sch (KiCad schematic)
At the start: 10 parts, among them J10 tp_ft232_, J11 tp_ft232_, J12 tp_ft232_, J13 tp_ft232_, J14 tp_ft232_, J7 tp_ft232_, J8 tp_ft232_, J9 tp_ft232_

Commit message: ESP32S3 branch initial changes
Parts:
- removed J14: tp_ft232_, Library:connector_pin1, symbol Connector:Conn_01x01_Pin
- removed JP1, JP2: SolderJumper_3_Bridged123, Jumper:SolderJumper-3_P1.3mm_Open_RoundedPad1.0x1.5mm_NumberLabels, symbol Jumper:SolderJumper_3_Bridged123
