File: usb_conector_Ft232.kicad_sch (KiCad schematic)
At the start: 9 parts, among them J4 tp_ft232_, J5 USB_B_Mini, J6 tp_ft232_, U4 LM1117DT-3.3

Commit message: ESP32S3 branch initial changes
Parts:
- removed J4: tp_ft232_, Library:connector_pin1, symbol Connector:Conn_01x01_Pin
- J5: footprint Library:USB_Mini-B_Wuerth_65100516121_Horizontal -> kiC:USB_Mini-B_Lumberg_2486_01_Horizontal
Changed lines of the file:
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@@
-	)
-	(junction
-		(at 132.08 83.82)
-		(diameter 0)
-		(color 0 0 0 0)
 	)
 	(junction
@@
 	(wire
 		(pts
-			(xy 127 83.82) (xy 132.08 83.82)
-		)
-		(stroke
-			(width 0)
-			(type default)
-		)
-	)
-	(wire
-		(pts
 			(xy 116.84 111.76) (xy 119.38 111.76)
 		)
@@
 	(wire
 		(pts
-			(xy 132.08 71.12) (xy 132.08 83.82)
-		)
-		(stroke
-			(width 0)
-			(type default)
-		)
-	)
-	(wire
-		(pts
 			(xy 175.26 93.98) (xy 162.56 93.98)
 		)
@@
 	(wire
 		(pts
-			(xy 127 83.82) (xy 127 92.71)
-		)
-		(stroke
-			(width 0)
-			(type default)
-		)
-	)
-	(wire
-		(pts
-			(xy 142.24 83.82) (xy 132.08 83.82)
+			(xy 135.89 83.82) (xy 135.89 92.71)
+		)
+		(stroke
+			(width 0)
+			(type default)
+		)
+	)
+	(wire
+		(pts
+			(xy 135.89 83.82) (xy 142.24 83.82)
 		)
 		(stroke
@@
 	(wire
 		(pts
-			(xy 120.65 71.12) (xy 132.08 71.12)
-		)
-		(stroke
-			(width 0)
-			(type default)
-		)
-	)
-	(wire
-		(pts
 			(xy 162.56 77.47) (xy 162.56 83.82)
 		)
@@
 		(pts
 			(xy 153.67 97.79) (xy 147.32 97.79)
+		)
+		(stroke
+			(width 0)
+			(type default)
+		)
+	)
+	(wire
+		(pts
+			(xy 135.89 92.71) (xy 127 92.71)
 		)
 		(stroke
@@
 			)
 		)
-		(property "Footprint" "Library:USB_Mini-B_Wuerth_65100516121_Horizontal"
+		(property "Footprint" "kiC:USB_Mini-B_Lumberg_2486_01_Horizontal"
 			(at 123.19 99.06 0)
 			(hide yes)
@@
 					(unit 1)
 				)
-			)
-		)
-	)
-	(symbol
-		(lib_id "Connector:Conn_01x01_Pin")
-		(at 115.57 71.12 0)
-		(mirror x)
-		(unit 1)
-		(body_style 1)
-		(exclude_from_sim no)
-		(in_bom yes)
-		(on_board yes)
-		(in_pos_files yes)
-		(dnp no)
-		(property "Reference" "J4"
-			(at 114.3 69.85 0)
-			(show_name no)
-			(do_not_autoplace no)
-			(effects
-				(font
-					(size 1.27 1.27)
-				)
-			)
-		)
-		(property "Value" "tp_ft232_"
-			(at 124.46 69.85 0)
-			(show_name no)
-			(do_not_autoplace no)
-			(effects
-				(font
-					(size 1.27 1.27)
-				)
-			)
-		)
-		(property "Footprint" "Library:connector_pin1"
-			(at 115.57 71.12 0)
-			(hide yes)
-			(show_name no)
-			(do_not_autoplace no)
-			(effects
-				(font
-					(size 1.27 1.27)
-				)
-			)
-		)
-		(property "Datasheet" ""
-			(at 115.57 71.12 0)
-			(hide yes)
-			(show_name no)
-			(do_not_autoplace no)
-			(effects
-				(font
-					(size 1.27 1.27)
-				)
-			)
-		)
-		(property "Description" ""
-			(at 115.57 71.12 0)
-			(show_name no)
-			(do_not_autoplace no)
-			(effects
-				(font
-					(size 1.27 1.27)
-				)
-			)
-		)
-		(pin "1"
-		)
-		(instances
-			(project "esp32_xiaozhi"
-				(path "/cae338e8-f342-43cb-b99a-a0486629133c/62520ce4-d21b-4842-a32d-5b11b343b2aa/78123daa-216c-4430-990d-f471f5bcbf11"
-					(reference "J4")
-					(unit 1)
-				)
