File: esp32_S3.kicad_sch (KiCad schematic)
At the start: 10 parts, among them SW9 boot, U5 ESP32-S3-WROOM-1, U8 ESP32-S3-DevKitC

Commit message: ESP32C6 branch changes
Parts:
- removed D10, D8, D9: LESD5D5.0CT1G, clackotron_fp:SOD-523_L1.2-W0.8-LS1.6-BI, symbol clackotronlib:LESD5D5.0CT1G
- removed D11: ESD3.3, Diode_SMD:D_SOD-923, symbol Diode:ESD9B3.3ST5G
- removed R30, R33: 5.1k, Resistor_SMD:R_0805_2012Metric, symbol Device:R
- removed SW9: boot, Button_Switch_SMD:SW_SPST_B3U-1000P, symbol Switch:SW_SPST
- removed U5: ESP32-S3-WROOM-1, Espressif:ESP32-S3-WROOM-1, symbol Espressif:ESP32-S3-WROOM-1
- removed U8: ESP32-S3-DevKitC, Espressif:ESP32-S3-DevKitC, symbol Espressif:ESP32-S3-DevKitC
- removed USBC1: USB3.1C16PFSMT, clackotron_fp:USB-C-SMD_TYPE-C-USB-17, symbol clackotronlib:USB3.1C16PFSMT
Connections:
- no-connect marks 2 -> 0
