File: power_supply.kicad_sch (KiCad schematic)
At the start: 5 parts

Commit message: ESP32S3 push before GPIO label changes
Parts:
- added C11, C3, C4: 100nf, Capacitor_SMD:C_0805_2012Metric, symbol Device:C
Connections:
- net +3V3: now also C11.1, C3.1, C4.1
- net GND: now also C11.2, C3.2, C4.2
