File: power_supply.kicad_sch (KiCad schematic)
At the start: 9 parts

Commit message: add files update
Parts:
- C32: value 100nf -> 1uf
Changed lines of the file:
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@@
 			)
 		)
-		(property "Value" "100nf"
+		(property "Value" "1uf"
 			(at 184.15 92.7099 0)
 			(hide yes)

Commit message: Actualización de esquemas y PCB con datos LCSC y librerías JLC
- Añade propiedades LCSC a los símbolos de las hojas de esquema
- Actualiza las hojas TXS0108E, display, esp32_c6, ft232, inmp441,
  led_sw_gpio, max98357a, micro_sd, power_supply y el esquema raíz
- Reorganiza el PCB (footprints, jumpers y nets) y actualiza el proyecto
- Incluye las librerías locales JLCImport (símbolos, huellas y modelos 3D)
  y las entradas correspondientes en fp-lib-table y sym-lib-table
- Añade la documentación técnica en docs/ y el archivo de posiciones
  esp32_xiaozhi-all.pos
- Elimina los ZIP generados gebers.zip y production.zip
Parts:
- C25, C26, C28, C29, C30, C31: LCSC (none) -> C1525
- C32: LCSC (none) -> C1848
- C53, C8: LCSC (none) -> C48587228
Changed lines of the file:
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@@
+			)
+		)
+		(property "LCSC" "C1525"
+			(at 123.19 130.81 0)
+			(hide yes)
+			(show_name no)
+			(do_not_autoplace no)
+			(effects
+				(font
+					(size 1.27 1.27)
+				)
 			)
 		)
@@
 			)
 		)
+		(property "LCSC" "C48587228"
+			(at 213.36 118.11 0)
+			(hide yes)
+			(show_name no)
+			(do_not_autoplace no)
+			(effects
+				(font
+					(size 1.27 1.27)
+				)
+			)
+		)
 		(pin "2"
 		)
@@
 			)
 		)
+		(property "LCSC" "C1525"
+			(at 137.16 130.81 0)
+			(hide yes)
+			(show_name no)
+			(do_not_autoplace no)
+			(effects
+				(font
+					(size 1.27 1.27)
+				)
+			)
+		)
 		(pin "1"
 		)
@@
 			)
 		)
+		(property "LCSC" "C1525"
+			(at 166.37 91.44 0)
+			(hide yes)
+			(show_name no)
+			(do_not_autoplace no)
+			(effects
+				(font
+					(size 1.27 1.27)
+				)
+			)
+		)
 		(pin "1"
 		)
@@
 			)
 		)
+		(property "LCSC" "C1525"
+			(at 151.13 130.81 0)
+			(hide yes)
+			(show_name no)
+			(do_not_autoplace no)
+			(effects
+				(font
+					(size 1.27 1.27)
+				)
+			)
+		)
 		(pin "1"
 		)
@@
 			)
 		)
+		(property "LCSC" "C1525"
+			(at 102.87 90.17 0)
+			(hide yes)
+			(show_name no)
+			(do_not_autoplace no)
+			(effects
+				(font
+					(size 1.27 1.27)
+				)
+			)
+		)
 		(pin "1"
 		)
@@
 			)
 		)
+		(property "LCSC" "C48587228"
+			(at 198.12 121.92 0)
+			(hide yes)
+			(show_name no)
+			(do_not_autoplace no)
+			(effects
+				(font
+					(size 1.27 1.27)
+				)
+			)
+		)
 		(pin "2"
 		)
@@
 			)
 		)
+		(property "LCSC" "C1848 "
+			(at 180.34 91.44 0)
+			(hide yes)
+			(show_name no)
+			(do_not_autoplace no)
+			(effects
+				(font
+					(size 1.27 1.27)
+				)
+			)
+		)
 		(pin "1"
 		)
@@
 			(show_name no)
 			(do_not_autoplace no)
+			(effects
+				(font
+					(size 1.27 1.27)
+				)
+			)
+		)
+		(property "LCSC" "C1525"
+			(at 88.9 90.17 0)
+			(hide yes)
+			(show_name no)
+			(do_not_autoplace no)

Commit message: add update
Parts:
- C25, C26, C28, C29, C31: LCSC C1525 -> C110255
- C30: value 100nf -> 1206B104K101NT; LCSC C1525 -> C110255
Changed lines of the file:
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@@
 			)
 		)
-		(property "LCSC" "C1525"
+		(property "LCSC" "C110255"
 			(at 123.19 130.81 0)
 			(hide yes)
@@
 			)
 		)
-		(property "LCSC" "C1525"
+		(property "LCSC" "C110255"
 			(at 137.16 130.81 0)
 			(hide yes)
@@
 			)
 		)
-		(property "LCSC" "C1525"
+		(property "LCSC" "C110255"
 			(at 166.37 91.44 0)
 			(hide yes)
@@
 			)
 		)
-		(property "Value" "100nf"
+		(property "Value" "1206B104K101NT"
 			(at 154.94 132.08 0)
 			(show_name no)
@@
 			)
 		)
-		(property "LCSC" "C1525"
+		(property "LCSC" "C110255"
 			(at 151.13 130.81 0)
 			(hide yes)
@@
 			)
 		)
-		(property "LCSC" "C1525"
+		(property "LCSC" "C110255"
 			(at 102.87 90.17 0)
 			(hide yes)
@@
 			)
 		)
-		(property "LCSC" "C1525"
+		(property "LCSC" "C110255"
 			(at 88.9 90.17 0)
 			(hide yes)

Commit message: correccion de partes
Parts:
- C53, C8: value 10uf -> RVT2A100M0607
Changed lines of the file:
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@@
 			)
 		)
-		(property "Value" "10uf"
+		(property "Value" "RVT2A100M0607"
 			(at 217.17 118.4909 0)
 			(show_name no)
@@
 			)
 		)
-		(property "Value" "10uf"
+		(property "Value" "RVT2A100M0607"
 			(at 201.93 122.3009 0)
 			(show_name no)
