File: Battery.kicad_sch (KiCad schematic)
At the start: 11 parts, among them U10 PCF85263ATL, Y1 Crystal

Commit message: ESP32S3: rename hierarchical GPIO labels and remove PCB tracks
Parts:
- removed BT1: Battery_Cell, JLCPCB:BAT-SMD_MYOUNG_MY-2032-04, symbol Device:Battery_Cell
- removed C5: 1uF, Capacitor_SMD:C_0805_2012Metric, symbol Device:C
- removed C6, C7, C8: 100nF, Capacitor_SMD:C_0805_2012Metric, symbol Device:C
- removed D7: WS2812B, LED_SMD:LED_WS2812B_PLCC4_5.0x5.0mm_P3.2mm, symbol LED:WS2812B
- removed R13, R14, R15: 10k, Resistor_SMD:R_0805_2012Metric, symbol Device:R
- removed U10: PCF85263ATL, Package_DFN_QFN:DFN-10-1EP_2.6x2.6mm_P0.5mm_EP1.3x2.2mm, symbol clackotronlib:PCF85263ATL
- removed Y1: Crystal, Crystal:Crystal_SMD_3215-2Pin_3.2x1.5mm, symbol Device:Crystal
Connections:
- no-connect marks 4 -> 0
