File: esp32_xiaozhi.kicad_pcb (KiCad board)
At the start: 2 copper layers, 99.1 x 99.1 mm, 70 parts, among them J21 conector oled ST1306 128x32, Q1 2N7002, SW1 power, SW2 up, SW3 down, SW4 left, SW5 rigth, U1 ESP32-WROOM-32, U2 TXS0108EPW, U3 FT232BM, U4 LM1117DT-3.3, U6 MAX98357A, Y2 6MHZ

Commit message: ESP32S3 branch initial changes
Parts:
- removed C23, C24, C25, C26, C32, C33, C34, C35, C9: 100nf, Capacitor_SMD:C_0805_2012Metric
- removed JP1, JP2: SolderJumper_3_Bridged123, Jumper:SolderJumper-3_P1.3mm_Open_RoundedPad1.0x1.5mm_NumberLabels
- removed the R12 at (137.3, 75.5)
- added C11: 100nf, Capacitor_SMD:C_0805_2012Metric, F.Cu at (88.1, 62.3)
- added C27: 100nf, Capacitor_SMD:C_0805_2012Metric, F.Cu at (49.4, 116.0)
- added C28: 100nf, Capacitor_SMD:C_0805_2012Metric, F.Cu at (33.9, 95.8)
- added C30: 22p, Capacitor_SMD:C_0805_2012Metric, F.Cu at (33.9, 98.8)
- added C37: 220p, Capacitor_SMD:C_0805_2012Metric, F.Cu at (33.9, 101.8)
- added C38: 10uf, Capacitor_SMD:C_0805_2012Metric, F.Cu at (33.9, 104.8)
- added C39: 100nf, Capacitor_SMD:C_0805_2012Metric, F.Cu at (177.8, 45.7)
- added C40: 100nf, Capacitor_SMD:C_0805_2012Metric, F.Cu at (177.8, 48.7)
- added C41: 100nf, Capacitor_SMD:C_0805_2012Metric, F.Cu at (177.8, 51.7)
- added D10: LESD5D5.0CT1G, clackotron_fp:SOD-523_L1.2-W0.8-LS1.6-BI, F.Cu at (95.5, 81.0)
- added D11: ESD3.3, Diode_SMD:D_SOD-923, F.Cu at (89.6, 85.8)
- added D3: LED, Diode_SMD:D_0805_2012Metric, F.Cu at (164.5, 142.0)
- added D4: LED, Diode_SMD:D_0805_2012Metric, F.Cu at (164.5, 139.0)
- added D5: LED, Diode_SMD:D_0805_2012Metric, F.Cu at (164.5, 135.9)
- added D6: LED, Diode_SMD:D_0805_2012Metric, F.Cu at (164.5, 132.9)
- added D7: WS2812B, LED_SMD:LED_WS2812B_PLCC4_5.0x5.0mm_P3.2mm, F.Cu at (198.6, 47.3)
- added D8: LESD5D5.0CT1G, clackotron_fp:SOD-523_L1.2-W0.8-LS1.6-BI, F.Cu at (95.5, 76.1)
- added D9: LESD5D5.0CT1G, clackotron_fp:SOD-523_L1.2-W0.8-LS1.6-BI, F.Cu at (95.5, 78.6)
- added J22: Adafruit ST7789, Library:Adafruit_SSD1306_No_Mounting_Holes_pads, F.Cu at (178.6, 99.0)
- added J5: USB_B_Mini, kiC:USB_Mini-B_Lumberg_2486_01_Horizontal, F.Cu at (97.8, 147.8)
- added L4: ferrite, Inductor_SMD:L_0805_2012Metric, F.Cu at (38.1, 102.2)
- added L5: ferrite, Inductor_SMD:L_0805_2012Metric, F.Cu at (38.1, 106.0)
- added L6: ferrite, Inductor_SMD:L_0805_2012Metric, F.Cu at (39.0, 128.5)
- added L7: ferrite, Inductor_SMD:L_0805_2012Metric, F.Cu at (39.0, 131.3)
- added R1: 2k2, Resistor_SMD:R_0805_2012Metric, F.Cu at (168.9, 141.7)
- added R14: 10k, Resistor_SMD:R_0805_2012Metric, F.Cu at (196.7, 39.6)
- added R15: 10k, Resistor_SMD:R_0805_2012Metric, F.Cu at (196.7, 42.5)
- added R2: 2k2, Resistor_SMD:R_0805_2012Metric, F.Cu at (168.9, 138.8)
- added R3: 2k2, Resistor_SMD:R_0805_2012Metric, F.Cu at (168.9, 135.8)
- added R33: 5.1k, Resistor_SMD:R_0805_2012Metric, F.Cu at (99.5, 79.3)
- added R34: 10K, Resistor_SMD:R_0805_2012Metric, F.Cu at (182.2, 42.2)
- added R36: 1M, Resistor_SMD:R_0805_2012Metric, F.Cu at (38.3, 95.8)
- added R37: 0, Jumper:SolderJumper-2_P1.3mm_Open_RoundedPad1.0x1.5mm, F.Cu at (38.3, 98.7)
- added R38: 1M, Resistor_SMD:R_0805_2012Metric, F.Cu at (47.8, 125.6)
- added R4: 2k2, Resistor_SMD:R_0805_2012Metric, F.Cu at (168.9, 132.9)
- added R5: 2k2, Resistor_SMD:R_0805_2012Metric, F.Cu at (64.5, 134.3)
- added R6: 2k2, Resistor_SMD:R_0805_2012Metric, F.Cu at (67.5, 134.3)
- added R7: 2k2, Resistor_SMD:R_0805_2012Metric, F.Cu at (70.4, 134.3)
- added R8: 2k2, Resistor_SMD:R_0805_2012Metric, F.Cu at (73.4, 134.3)
- added SW2: down, Button_Switch_SMD:SW_Push_1P1T_NO_CK_KSC9xxG, F.Cu at (68.5, 142.0)
- added SW3: left, Button_Switch_SMD:SW_Push_1P1T_NO_CK_KSC9xxG, F.Cu at (76.0, 142.0)
- added SW4: rigth, Button_Switch_SMD:SW_Push_1P1T_NO_CK_KSC9xxG, F.Cu at (83.4, 142.0)
- added SW9: boot, Button_Switch_SMD:SW_SPST_B3U-1000P, F.Cu at (85.3, 87.0)
- added U10: PCF85263ATL, Package_DFN_QFN:DFN-10-1EP_2.6x2.6mm_P0.5mm_EP1.3x2.2mm, F.Cu at (201.8, 37.2)
- added U5: ESP32-S3-WROOM-1, Espressif:ESP32-S3-WROOM-1, F.Cu at (68.9, 63.8)
- added U7: ER_OLEDM0.91_1x-I2C, Connector_PinHeader_2.54mm:PinHeader_1x04_P2.54mm_Vertical, F.Cu at (132.7, 58.1)
- added U8: ESP32-S3-DevKitC, Espressif:ESP32-S3-DevKitC, F.Cu at (57.4, 54.7)
- added U9: ESP32-C6-WROOM-1-N8, kiC:XCVR_ESP32-C6-WROOM-1-N8, F.Cu at (105.8, 60.1)
- added USBC1: USB3.1C16PFSMT, clackotron_fp:USB-C-SMD_TYPE-C-USB-17, F.Cu at (59.7, 124.7)
- added Y1: Crystal, Crystal:Crystal_SMD_3215-2Pin_3.2x1.5mm, F.Cu at (201.5, 41.0)
- C5: value 100nf -> 1uF
- C6, C7, C8: value 100nf -> 100nF
- J21: value conector oled ST1306 128x32 -> Oled SSD1306 128x32
- R13: value 2k2 -> 10k
- R30: value 10K -> 5.1k
- R31, R32: value 1k -> 2k2
- SW1: value power -> up; footprint Button_Switch_SMD:SW_SPST_CK_RS282G05A3 -> Button_Switch_SMD:SW_Push_1P1T_NO_CK_KSC9xxG
- SW5: renamed from SW2; footprint Button_Switch_SMD:SW_SPST_CK_RS282G05A3 -> Button_Switch_SMD:SW_Push_1P1T_NO_CK_KSC9xxG
- SW6: renamed from SW3; footprint Button_Switch_SMD:SW_SPST_CK_RS282G05A3 -> Button_Switch_SMD:SW_Push_1P1T_NO_CK_KSC9xxG
- SW7: renamed from SW4; footprint Button_Switch_SMD:SW_SPST_CK_RS282G05A3 -> Button_Switch_SMD:SW_Push_1P1T_NO_CK_KSC9xxG
- SW8: renamed from SW5; footprint Button_Switch_SMD:SW_SPST_CK_RS282G05A3 -> Button_Switch_SMD:SW_Push_1P1T_NO_CK_KSC9xxG
- U1: value ESP32-WROOM-32 -> ESP32-C6-DEVKITC-1-N8; footprint RF_Module:ESP32-WROOM-32 -> kiC:MODULE_ESP32-C6-DEVKITC-1-N8
- moved C5 132.0 mm to (192.3, 36.7)
- moved C6 132.0 mm to (192.3, 39.7)
- moved D1 123.2 mm to (198.4, 77.9)
- moved D2 123.2 mm to (198.4, 81.0)
- moved R24 123.2 mm to (195.8, 61.6)
- moved R25 123.2 mm to (195.8, 64.6)
- moved R26 123.2 mm to (195.8, 67.5)
- moved R27 123.2 mm to (195.8, 70.5)
- moved C16 123.2 mm to (200.2, 61.7)
- moved C17 123.2 mm to (200.2, 64.7)
- moved C18 123.2 mm to (200.2, 67.7)
- moved R16 123.2 mm to (187.0, 61.6)
- moved R17 123.2 mm to (187.0, 64.6)
- moved R18 123.2 mm to (187.0, 67.5)
- moved R19 123.2 mm to (187.0, 70.5)
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- renumbered R11 to R10, R14 to R11, R15 to R12, R10 to R9
Connections:
- net /display/scl renamed /display/SCL
- net /display/sda renamed /display/SDA
- net /led_sw_gpio/RD4 renamed /led_sw_gpio/sw5
- net /led_sw_gpio/RD5 renamed /led_sw_gpio/sw6
- net /led_sw_gpio/RD6 renamed /led_sw_gpio/sw7
- net /led_sw_gpio/RD7 renamed /led_sw_gpio/sw8
- net Net-(U6-GND-Pad11) renamed GNDA
- C1 pad 1: +3.3V -> +3V3
- C10 pad 1: +3.3V -> +3V3
- C2 pad 1: +3.3V -> +3V3
- C3 pad 1: +3.3V -> +3V3
- C36 pad 1: +5V -> +3V3
- C4 pad 1: +3.3V -> +3V3
- C5 pad 1: +3.3V -> +3V3
- C6 pad 1: +3.3V -> Net-(BT1-+)
- C7 pad 1: +3.3V -> +5V
- C8 pad 1: +3.3V -> +3V3
- J21 pad 1: GND -> +3.3V
- J21 pad 2: +3.3V -> +5V
- J21 pad 4: /display/RG7 -> +5V
- J21 pad 6: /display/RG8 -> GND
- MK1 pad 1: unconnected-(MK1-SCK-Pad1) -> /inmp441/SCK
- MK1 pad 2: unconnected-(MK1-SD-Pad2) -> /inmp441/SD
- MK1 pad 3: unconnected-(MK1-WS-Pad3) -> /inmp441/WS
- MK1 pad 4: unconnected-(MK1-L/R-Pad4) -> /inmp441/L/R
- MK1 pad 7: unconnected-(MK1-VDD-Pad7) -> Net-(MK1-VDD)
- MK1 pad 8: unconnected-(MK1-CHIPEN-Pad8) -> /inmp441/EN
- R10 pad 1: +3.3V -> +3V3
- R11 pad 1: +3.3V -> +3V3
- R12 pad 1: +3.3V -> +3V3
- R13 pad 1: SW_PWR -> Net-(U10-OSCI)
- R13 pad 2: GND -> Net-(R13-Pad2)
- R20 pad 2: /ft232/RX_MCU -> /ft232/FT_TX
- R21 pad 2: /ft232/TX_MCU -> /ft232/FT_RX
- R30 pad 1: +3V3 -> GND
- R30 pad 2: /ft232/FT_RESET -> Net-(USBC1-CC2)
- R31 pad 1: +3.3V -> +3V3
- R32 pad 1: +3.3V -> +3V3
- R9 pad 1: +3.3V -> +3V3
- SW1 pad 1: Net-(R12-Pad2) -> /led_sw_gpio/sw1
- SW1 pad 2: SW_PWR -> GND
- U2 pad 1: unconnected-(U2-A1-Pad1) -> /TXS0108E/A1
- U2 pad 10: unconnected-(U2-OE-Pad10) -> /TXS0108E/OE
- U2 pad 11: unconnected-(U2-GND-Pad11) -> GND
- U2 pad 12: unconnected-(U2-B8-Pad12) -> /TXS0108E/B8
- U2 pad 13: unconnected-(U2-B7-Pad13) -> /TXS0108E/B7
- U2 pad 14: unconnected-(U2-B6-Pad14) -> /TXS0108E/B6
- U2 pad 15: unconnected-(U2-B5-Pad15) -> /TXS0108E/B5
- U2 pad 16: unconnected-(U2-B4-Pad16) -> /TXS0108E/B4
- U2 pad 17: unconnected-(U2-B3-Pad17) -> /TXS0108E/B3
- U2 pad 18: unconnected-(U2-B2-Pad18) -> /TXS0108E/B2
- U2 pad 19: unconnected-(U2-VCCB-Pad19) -> +5V
- U2 pad 2: unconnected-(U2-VCCA-Pad2) -> +3V3
- U2 pad 20: unconnected-(U2-B1-Pad20) -> /TXS0108E/B1
- U2 pad 3: unconnected-(U2-A2-Pad3) -> /TXS0108E/A2
- U2 pad 4: unconnected-(U2-A3-Pad4) -> /TXS0108E/A3
- U2 pad 5: unconnected-(U2-A4-Pad5) -> /TXS0108E/A4
- U2 pad 6: unconnected-(U2-A5-Pad6) -> /TXS0108E/A5
- U2 pad 7: unconnected-(U2-A6-Pad7) -> /TXS0108E/A6
- U2 pad 8: unconnected-(U2-A7-Pad8) -> /TXS0108E/A7
- U2 pad 9: unconnected-(U2-A8-Pad9) -> /TXS0108E/A8
- U3 pad 23: /ft232/FT_RESET -> /ft232/FT_RST
- U6 pad 1: unconnected-(U6-DIN-Pad1) -> /max98357a/DIN
- U6 pad 10: unconnected-(U6-OUTN-Pad10) -> /max98357a/OUTN
- U6 pad 14: unconnected-(U6-LRCLK-Pad14) -> /max98357a/LRC
- U6 pad 16: unconnected-(U6-BCLK-Pad16) -> /max98357a/BCLK
- U6 pad 17: unconnected-(U6-PAD-Pad17) -> /max98357a/pad
- U6 pad 2: unconnected-(U6-GAIN_SLOT-Pad2) -> /max98357a/GAIN
- U6 pad 4: unconnected-(U6-~{SD_MODE}-Pad4) -> /max98357a/SD
- U6 pad 9: unconnected-(U6-OUTP-Pad9) -> /max98357a/OUTP

Commit message: Update KiCad project files
Parts:
- removed the C11 at (88.1, 62.3)
- removed the C19 at (208.3, 58.6)
- removed the C20 at (208.3, 61.6)
- removed the C4 at (88.1, 59.3)
- removed the C5 at (192.3, 36.7)
- removed the C6 at (192.3, 39.7)
- removed the C7 at (192.3, 42.7)
- removed C8: 100nF, Capacitor_SMD:C_0805_2012Metric
- removed D10, D8, D9: LESD5D5.0CT1G, clackotron_fp:SOD-523_L1.2-W0.8-LS1.6-BI
- removed D11: ESD3.3, Diode_SMD:D_SOD-923
- removed the L2 at (217.8, 58.9)
- removed L6: ferrite, Inductor_SMD:L_0805_2012Metric
- removed the R13 at (196.7, 36.6)
- removed the R14 at (196.7, 39.6)
- removed the R28 at (212.7, 58.6)
- removed the R29 at (212.7, 61.6)
- removed the R30 at (99.5, 76.4)
- removed the R33 at (99.5, 79.3)
- removed the SW9 at (85.3, 87.0)
- removed U10: PCF85263ATL, Package_DFN_QFN:DFN-10-1EP_2.6x2.6mm_P0.5mm_EP1.3x2.2mm
- removed the U5 at (68.9, 63.8)
- removed U8: ESP32-S3-DevKitC, Espressif:ESP32-S3-DevKitC
- removed U9: ESP32-C6-WROOM-1-N8, kiC:XCVR_ESP32-C6-WROOM-1-N8
- removed USBC1: USB3.1C16PFSMT, clackotron_fp:USB-C-SMD_TYPE-C-USB-17
- removed Y2: 6MHZ, Crystal:Crystal_SMD_0603-4Pin_6.0x3.5mm
- added C1: 100nf, Capacitor_SMD:C_0805_2012Metric, F.Cu at (212.9, 86.1)
- added C13: 100n, Capacitor_SMD:C_0402_1005Metric, F.Cu at (167.7, 120.5)
- added C14: 100n, Capacitor_SMD:C_0402_1005Metric, F.Cu at (167.7, 116.6)
- added C17: 100nf, Capacitor_SMD:C_0805_2012Metric, F.Cu at (99.3, 122.7)
- added C18: 100nf, Capacitor_SMD:C_0805_2012Metric, F.Cu at (116.3, 133.1)
- added C2: 100nf, Capacitor_SMD:C_0805_2012Metric, F.Cu at (212.9, 89.1)
- added C22: 220p, Capacitor_SMD:C_0805_2012Metric, F.Cu at (139.0, 101.9)
- added C24: 100nF, Capacitor_SMD:C_0805_2012Metric, F.Cu at (139.9, 86.1)
- added C27: 100nf, Capacitor_SMD:C_0805_2012Metric, F.Cu at (53.1, 112.9)
- added C28: 100nf, Capacitor_SMD:C_0805_2012Metric, F.Cu at (145.9, 110.7)
- added C29: 100nf, Capacitor_SMD:C_0805_2012Metric, F.Cu at (98.3, 62.0)
- added C30: 100nf, Capacitor_SMD:C_0805_2012Metric, F.Cu at (112.2, 109.3)
- added C33: 100nf, Capacitor_SMD:C_0805_2012Metric, F.Cu at (53.1, 115.9)
- added C34: 100nf, Capacitor_SMD:C_0805_2012Metric, F.Cu at (53.1, 104.9)
- added C35: 100nf, Capacitor_SMD:C_0805_2012Metric, F.Cu at (53.1, 107.9)
- added C36: 100nf, Capacitor_SMD:C_0805_2012Metric, F.Cu at (43.7, 104.9)
- added C38: 100nf, Capacitor_SMD:C_0805_2012Metric, F.Cu at (43.7, 110.9)
- added J1: FT232RL, Connector_PinHeader_2.54mm:PinHeader_1x06_P2.54mm_Vertical, F.Cu at (74.5, 131.4)
- added J10: Micro_SD_Card, Library:3M_2908-05WB-MG, F.Cu at (146.8, 122.7)
- added J3: USB_B_Mini, kiC:USB_Mini-B_Lumberg_2486_01_Horizontal, F.Cu at (106.5, 147.2)
- added J6: Conn_01x03_Pin, Connector_PinHeader_2.54mm:PinHeader_1x03_P2.54mm_Vertical, F.Cu at (109.8, 103.4)
- added J7: Conn_01x07_Pin, Connector_PinHeader_2.54mm:PinHeader_1x07_P2.54mm_Vertical, F.Cu at (134.5, 93.3)
- added JP1: Jumper_2_Open, Jumper:SolderJumper-2_P1.3mm_Open_RoundedPad1.0x1.5mm, F.Cu at (88.7, 122.0)
- added JP2: Jumper_2_Open, Jumper:SolderJumper-2_P1.3mm_Bridged_RoundedPad1.0x1.5mm, F.Cu at (161.6, 131.2)
- added JP3: Jumper_2_Open, Jumper:SolderJumper-2_P1.3mm_Open_RoundedPad1.0x1.5mm, F.Cu at (161.6, 134.8)
- added JP4: Jumper_2_Open, Jumper:SolderJumper-2_P1.3mm_Open_RoundedPad1.0x1.5mm, F.Cu at (161.6, 138.3)
- added JP5: NL, Jumper:SolderJumper-2_P1.3mm_Open_RoundedPad1.0x1.5mm, F.Cu at (87.9, 102.9)
- added JP6: NL, Jumper:SolderJumper-2_P1.3mm_Open_RoundedPad1.0x1.5mm, F.Cu at (87.9, 106.4)
- added L1: 100mh, Inductor_SMD:L_1206_3216Metric, F.Cu at (102.2, 140.1)
- added LS1: Speaker, Connector_Molex:Molex_Micro-Latch_53253-0270_1x02_P2.00mm_Vertical, F.Cu at (149.5, 89.6)
- added Q10: FDN306P, Package_TO_SOT_SMD:SOT-23W, F.Cu at (39.1, 102.1)
- added Q11: FDN306P, Package_TO_SOT_SMD:SOT-23W, F.Cu at (92.6, 103.5)
- added Q4: Q_NPN_BCE, Package_TO_SOT_SMD:SOT-23W, F.Cu at (163.8, 109.1)
- added Q5: Q_NPN_BCE, Package_TO_SOT_SMD:SOT-23W, F.Cu at (163.8, 113.9)
- added Q6: 2N7002, Package_TO_SOT_SMD:SOT-23, F.Cu at (152.8, 80.5)
- added Q7: Q_NPN_BCE, Package_TO_SOT_SMD:SOT-23W, F.Cu at (39.0, 105.8)
- added Q8: Q_NPN_BCE, Package_TO_SOT_SMD:SOT-23W, F.Cu at (39.0, 110.6)
- added Q9: 2N7002, Package_TO_SOT_SMD:SOT-23, F.Cu at (43.9, 114.6)
- added R16: 10k, Resistor_SMD:R_0402_1005Metric, F.Cu at (174.3, 109.7)
- added R20: 10k, Resistor_SMD:R_0402_1005Metric, F.Cu at (174.3, 111.7)
- added R22: 27, Resistor_SMD:R_0805_2012Metric, F.Cu at (108.8, 140.4)
- added R23: 27, Resistor_SMD:R_0805_2012Metric, F.Cu at (106.1, 140.4)
- added R38: 2k2, Resistor_SMD:R_0805_2012Metric, F.Cu at (148.2, 79.8)
- added R40: 2k2, Resistor_SMD:R_0805_2012Metric, F.Cu at (148.2, 82.7)
- added R43: 4k7, Resistor_SMD:R_0805_2012Metric, F.Cu at (135.6, 115.3)
- added R44: 4k7, Resistor_SMD:R_0805_2012Metric, F.Cu at (135.6, 118.3)
- added R45: 4k7, Resistor_SMD:R_0805_2012Metric, F.Cu at (135.6, 121.2)
- added R46: 4k7, Resistor_SMD:R_0805_2012Metric, F.Cu at (135.6, 124.2)
- added R47: 4k7, Resistor_SMD:R_0805_2012Metric, F.Cu at (135.6, 127.1)
- added R48: 4k7, Resistor_SMD:R_0805_2012Metric, F.Cu at (135.6, 130.1)
- added R49: 10k, Resistor_SMD:R_0603_1608Metric, F.Cu at (47.4, 104.4)
- added R50: 10k, Resistor_SMD:R_0603_1608Metric, F.Cu at (47.4, 106.4)
- added R51: 10k, Resistor_SMD:R_0603_1608Metric, F.Cu at (47.4, 108.4)
- added R52: 10k, Resistor_SMD:R_0603_1608Metric, F.Cu at (47.4, 110.4)
- added R53: 10k, Resistor_SMD:R_0603_1608Metric, F.Cu at (92.1, 107.1)
- added SW1: SW_Push, Button_Switch_SMD:SW_Push_SPST_NO_Alps_SKRK, F.Cu at (169.5, 108.9)
- added SW2: SW_Push, Button_Switch_SMD:SW_Push_SPST_NO_Alps_SKRK, F.Cu at (169.5, 113.4)
- added U2: ESP32-C6-DEVKITC-1-N8, kiC:MODULE_ESP32-C6-DEVKITC-1-N8, F.Cu at (71.1, 80.0)
- C10: value 100nf -> 100n; footprint Capacitor_SMD:C_0805_2012Metric -> Capacitor_SMD:C_0402_1005Metric
- C37: value 220p -> 100nf
- J5: value USB_B_Mini -> Conn_01x03_Pin; footprint kiC:USB_Mini-B_Lumberg_2486_01_Horizontal -> Connector_PinHeader_2.54mm:PinHeader_1x03_P2.54mm_Vertical
- R15: footprint Resistor_SMD:R_0805_2012Metric -> Resistor_SMD:R_0402_1005Metric
- U1: value ESP32-C6-DEVKITC-1-N8 -> ESP32-C6-WROOM-1-N8; footprint kiC:MODULE_ESP32-C6-DEVKITC-1-N8 -> kiC:XCVR_ESP32-C6-WROOM-1-N8
- Y1: footprint Crystal:Crystal_SMD_3215-2Pin_3.2x1.5mm -> Crystal:Resonator-2Pin_W10.0mm_H5.0mm
- moved U4 150.5 mm to (94.2, 145.5), turned to 90 degrees
- moved Y1 138.1 mm to (94.6, 128.4)
- moved C3 129.9 mm to (212.9, 92.1)
- moved C15 127.1 mm to (95.2, 133.2), turned to 180 degrees
- moved C6 125.5 mm to (98.9, 146.3), turned to 90 degrees
- moved C5 124.3 mm to (95.1, 138.5), turned to 90 degrees
- moved R18 123.2 mm to (100.0, 134.0)
- moved C16 117.4 mm to (95.2, 123.1), turned to 180 degrees
- moved R21 116.0 mm to (100.6, 136.9)
- moved C20 114.6 mm to (148.4, 100.4), turned to -90 degrees
- moved C23 114.3 mm to (148.1, 97.0)
- moved R17 114.1 mm to (108.1, 137.6)
- moved C12 113.8 mm to (113.2, 141.1)
- moved C7 113.7 mm to (115.8, 147.1), turned to 90 degrees
- moved L4 108.6 mm to (146.7, 106.0)
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- renumbered C17 to C11, C18 to C12, C21 to C15, C22 to C16, C27 to C19, C28 to C20, C38 to C21, C30 to C23, C1 to C25, C2 to C26, C29 to C31, C31 to C32, C36 to C4, C39 to C5, C40 to C6, C41 to C7, C16 to C9, J21 to J8, J22 to J9, L7 to L2, L4 to L3, L5 to L4, Q1 to Q2, R20 to R10, R21 to R11, R22 to R12, R23 to R13, R24 to R14, R25 to R17, R34 to R18, R26 to R19, R16 to R2, R27 to R21, R38 to R24, R36 to R25, R37 to R26, R1 to R27, R2 to R28, R3 to R29, R4 to R30, R5 to R31, R6 to R32, R7 to R33, R8 to R34, R9 to R35, R10 to R36, R11 to R37, R12 to R39, R31 to R41, R32 to R42, R17 to R6, R18 to R7, R19 to R8, SW8 to SW10, SW1 to SW3, SW2 to SW4, SW3 to SW5, SW4 to SW6, SW5 to SW7, SW6 to SW8, SW7 to SW9, U6 to U5, U7 to U6, U2 to U7
Connections:
- net /TXS0108E/A1 renamed /Logic_convert/A1
- net /TXS0108E/A2 renamed /Logic_convert/A2
- net /TXS0108E/A3 renamed /Logic_convert/A3
- net /TXS0108E/A4 renamed /Logic_convert/A4
- net /TXS0108E/A5 renamed /Logic_convert/A5
- net /TXS0108E/A6 renamed /Logic_convert/A6
- net /TXS0108E/A7 renamed /Logic_convert/A7
- net /TXS0108E/A8 renamed /Logic_convert/A8
- net /TXS0108E/B1 renamed /Logic_convert/B1
- net /TXS0108E/B2 renamed /Logic_convert/B2
- net /TXS0108E/B3 renamed /Logic_convert/B3
- net /TXS0108E/B4 renamed /Logic_convert/B4
- net /TXS0108E/B5 renamed /Logic_convert/B5
- net /TXS0108E/B6 renamed /Logic_convert/B6
- net /TXS0108E/B7 renamed /Logic_convert/B7
- net /TXS0108E/B8 renamed /Logic_convert/B8
- net /max98357a/pad renamed /max98357a/PAD
- C10 pad 1: +3V3 -> /ft232/EN
- C37 pad 1: GNDA -> +3V3
- C37 pad 2: Net-(C37-Pad2) -> GND
- D3 pad 1: +3V3 -> /led_sw_gpio/led3
- D4 pad 1: +3V3 -> /led_sw_gpio/led4
- D5 pad 1: +3V3 -> /led_sw_gpio/led5
- D6 pad 1: +3V3 -> /led_sw_gpio/led6
- J5 pad 1: Net-(J5-VBUS) -> /inmp441/SCK
- J5 pad 2: Net-(J5-D-) -> /inmp441/EN
- J5 pad 3: Net-(J5-D+) -> /inmp441/L/R
- L2 pad 2: +5V -> Net-(JP3-A)
- R15 pad 1: +3V3 -> /ft232/FT_DTR
- R15 pad 2: SDA -> Net-(Q4-B)
- U7 pad 10: /TXS0108E/OE -> /Logic_convert/OEN
- Y1 pad 1: Net-(R13-Pad2) -> /ft232/FT_XTIN
- Y1 pad 2: Net-(U10-OSCO) -> /ft232/FT_XTOUT
Routing:
- net Net-(U3-AVCC): vias 0 -> 2
- net Net-(D2-K): vias 0 -> 2
- net Net-(C22-Pad2): vias 0 -> 1
- net GND: vias 0 -> 2
- net /ft232/V+_USB: vias 0 -> 3
- net /ft232/FT_RESET: vias 0 -> 2
- net +3V3: vias 0 -> 6

Commit message: Remove all vias from PCB
Parts:
- removed J6: Conn_01x03_Pin, Connector_PinHeader_2.54mm:PinHeader_1x03_P2.54mm_Vertical
- removed J8: Oled SSD1306 128x32, Connector_PinHeader_2.54mm:PinHeader_2x03_P2.54mm_Vertical
- removed R24: 1M, Resistor_SMD:R_0805_2012Metric
- removed R26: 0, Jumper:SolderJumper-2_P1.3mm_Open_RoundedPad1.0x1.5mm
- added JP7: 0, Jumper:SolderJumper-2_P1.3mm_Open_RoundedPad1.0x1.5mm, F.Cu at (142.9, 93.3)
- added L5: ferrite, Inductor_SMD:L_0805_2012Metric, F.Cu at (152.7, 96.6)
- added L6: ferrite, Inductor_SMD:L_0805_2012Metric, F.Cu at (152.7, 99.4)
- added MK2: INMP441ACEZ-R7, kiC:MODULE_OKY3139, F.Cu at (220.0, 133.0)
- J5: value Conn_01x03_Pin -> Oled SSD1306 128x32; footprint Connector_PinHeader_2.54mm:PinHeader_1x03_P2.54mm_Vertical -> Connector_PinHeader_2.54mm:PinHeader_2x03_P2.54mm_Vertical
- JP2: footprint Jumper:SolderJumper-2_P1.3mm_Bridged_RoundedPad1.0x1.5mm -> Jumper:SolderJumper-2_P1.3mm_Open_RoundedPad1.0x1.5mm
- U6: footprint Connector_PinHeader_2.54mm:PinHeader_1x04_P2.54mm_Vertical -> kiC:LCD_OLED_128X64_1.3_I2C
- moved L2 122.0 mm to (219.9, 129.0)
- moved C19 120.6 mm to (220.0, 136.9)
- moved MK1 117.2 mm to (220.0, 133.0), turned to -90 degrees
- moved J5 69.9 mm to (168.4, 133.2)
- moved JP4 63.2 mm to (223.6, 126.2), turned to 90 degrees
- moved JP3 59.1 mm to (220.0, 126.0), turned to 90 degrees
- moved Q6 57.9 mm to (100.3, 105.0), turned to 90 degrees
- moved R38 56.6 mm to (97.2, 104.4), turned to 90 degrees
- moved JP2 55.1 mm to (216.5, 126.1), turned to 90 degrees
- moved R40 52.6 mm to (98.7, 100.5), turned to 90 degrees
- moved D7 52.0 mm to (98.7, 110.4)
- moved R14 18.7 mm to (98.6, 140.3), turned to -90 degrees
- moved U6 15.5 mm to (136.0, 73.7), turned to 0 degrees
- moved C15 5.88 mm to (92.3, 128.2), turned to -90 degrees
- moved R18 4.31 mm to (96.9, 137.0)
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Connections:
- net Net-(J6-Pin_3) renamed /inmp441/VDD_INMP441
- C20 pad 2: Net-(J7-Pin_3) -> /max98357a/VCC_MAC98357
- C21 pad 2: Net-(J7-Pin_3) -> /max98357a/VCC_MAC98357
- J5 pad 1: /inmp441/SCK -> +3.3V
- J5 pad 2: /inmp441/EN -> +5V
- J5 pad 3: /inmp441/L/R -> /display/SDA
- J7 pad 1: /max98357a/GAIN -> /max98357a/LRC
- J7 pad 2: /max98357a/SD -> /max98357a/BCLK
- J7 pad 3: Net-(J7-Pin_3) -> /max98357a/DIN
- J7 pad 4: /max98357a/LRC -> /max98357a/GAIN
- J7 pad 5: /max98357a/BCLK -> /max98357a/SD
- J7 pad 6: /max98357a/DIN -> GNDA
- J7 pad 7: GNDA -> /max98357a/VCC_MAC98357
- L3 pad 1: Net-(J7-Pin_3) -> /max98357a/VCC_MAC98357
- L4 pad 1: Net-(J7-Pin_3) -> /max98357a/VCC_MAC98357
- U5 pad 7: Net-(J7-Pin_3) -> /max98357a/VCC_MAC98357
- U5 pad 8: Net-(J7-Pin_3) -> /max98357a/VCC_MAC98357
Routing:
- net Net-(U3-AVCC): vias 2 -> 0
- net Net-(D2-K): vias 2 -> 0
- net Net-(C22-Pad2): vias 1 -> 0
- net GND: vias 2 -> 0
- net /ft232/V+_USB: vias 3 -> 0
- net /ft232/FT_RESET: vias 2 -> 0
- net +3V3: vias 6 -> 0
