File: esp32_xiaozhi.kicad_pcb (KiCad board)
At the start: 2 copper layers, 27 parts, among them J13 tp, J20 tp, SW11 boot, SW3 up, SW4 down, U6 ER_OLEDM0.91_1x-I2C, Y1 Crystal

Commit message: Update all schematic files and project
Parts:
- added C1: 100nf, Capacitor_SMD:C_0805_2012Metric, F.Cu at (87.9, 57.8)
- added C10: 100n, Capacitor_SMD:C_0805_2012Metric, F.Cu at (83.4, 111.3)
- added C11: 33nf, Capacitor_SMD:C_0805_2012Metric, F.Cu at (94.6, 141.0)
- added C13: 100n, Capacitor_SMD:C_0805_2012Metric, F.Cu at (163.2, 119.5)
- added C14: 100n, Capacitor_SMD:C_0805_2012Metric, F.Cu at (102.9, 100.5)
- added C16: 15p, Capacitor_SMD:C_0805_2012Metric, F.Cu at (97.0, 132.2)
- added C19: 100nf, Capacitor_SMD:C_0805_2012Metric, F.Cu at (122.2, 108.5)
- added C2: 100nf, Capacitor_SMD:C_0805_2012Metric, F.Cu at (81.3, 122.2)
- added C21: 10uf, Capacitor_SMD:C_0805_2012Metric, F.Cu at (139.3, 111.1)
- added C22: 220p, Capacitor_SMD:C_0805_2012Metric, F.Cu at (147.6, 106.0)
- added C23: 22p, Capacitor_SMD:C_0805_2012Metric, F.Cu at (145.6, 110.2)
- added C24: 100nF, Capacitor_SMD:C_0805_2012Metric, F.Cu at (92.7, 71.9)
- added C25: 100nf, Capacitor_SMD:C_1206_3216Metric, F.Cu at (132.2, 63.4)
- added C26: 100nf, Capacitor_SMD:C_1206_3216Metric, F.Cu at (91.2, 62.2)
- added C27: 100nf, Capacitor_SMD:C_0805_2012Metric, F.Cu at (98.3, 65.0)
- added C28: 100nf, Capacitor_SMD:C_1206_3216Metric, F.Cu at (147.8, 113.5)
- added C29: 100nf, Capacitor_SMD:C_1206_3216Metric, F.Cu at (98.3, 62.0)
- added C3: 100nf, Capacitor_SMD:C_0805_2012Metric, F.Cu at (127.9, 89.0)
- added C30: 100nf, Capacitor_SMD:C_1206_3216Metric, F.Cu at (122.7, 76.5)
- added C31: 100nf, Capacitor_SMD:C_1206_3216Metric, F.Cu at (141.4, 113.4)
- added C32: 100nf, Capacitor_SMD:C_1206_3216Metric, F.Cu at (144.4, 63.4)
- added C33: 100nf, Capacitor_SMD:C_0805_2012Metric, F.Cu at (60.9, 132.4)
- added C34: 100nf, Capacitor_SMD:C_0805_2012Metric, F.Cu at (143.1, 87.3)
- added C35: 100nf, Capacitor_SMD:C_0805_2012Metric, F.Cu at (148.0, 67.9)
- added C36: 100nf, Capacitor_SMD:C_0805_2012Metric, F.Cu at (104.4, 64.9)
- added C37: 100nf, Capacitor_SMD:C_0805_2012Metric, F.Cu at (104.2, 68.0)
- added C38: 100nf, Capacitor_SMD:C_0805_2012Metric, F.Cu at (92.8, 66.6)
- added C39: 100nf, Capacitor_SMD:C_0805_2012Metric, F.Cu at (78.3, 136.8)
- added C40: 100nf, Capacitor_SMD:C_0805_2012Metric, F.Cu at (61.7, 145.0)
- added C41: 100nf, Capacitor_SMD:C_0805_2012Metric, F.Cu at (133.4, 138.0)
- added C42: 100nf, Capacitor_SMD:C_0805_2012Metric, F.Cu at (78.3, 138.9)
- added C43: 100nf, Capacitor_SMD:C_0805_2012Metric, F.Cu at (133.4, 133.4)
- added C44: 100nf, Capacitor_SMD:C_0805_2012Metric, F.Cu at (138.5, 134.8)
- added C45: 100nf, Capacitor_SMD:C_1206_3216Metric, F.Cu at (74.5, 100.4)
- added C47: 100nf, Capacitor_SMD:C_0805_2012Metric, F.Cu at (118.2, 134.9)
- added C48: 100nf, Capacitor_SMD:C_0805_2012Metric, F.Cu at (118.6, 139.0)
- added C49: 100nf, Capacitor_SMD:C_1206_3216Metric, F.Cu at (172.4, 119.7)
- added C5: 100nf, Capacitor_SMD:C_0805_2012Metric, B.Cu at (95.7, 137.7)
- added C50: 100n, Capacitor_SMD:C_0805_2012Metric, F.Cu at (163.2, 122.5)
- added C51: 100n, Capacitor_SMD:C_0805_2012Metric, F.Cu at (163.2, 125.5)
- added C9: 100nf, Capacitor_SMD:C_0805_2012Metric, F.Cu at (104.3, 122.8)
- added D1: RX, Diode_SMD:D_0805_2012Metric, F.Cu at (116.1, 139.2)
- added D11: LESD5D5.0CT1G, Diode_SMD:D_SOD-523, F.Cu at (65.2, 119.0)
- added D12: ESD3.3, Diode_SMD:D_SOD-923, F.Cu at (77.5, 111.7)
- added D13: LED, Diode_SMD:D_0805_2012Metric, F.Cu at (179.5, 125.4)
- added D14: 1N5819, Diode_SMD:D_2512_6332Metric, F.Cu at (165.4, 115.5)
- added D2: RX, Diode_SMD:D_0805_2012Metric, F.Cu at (113.8, 138.8)
- added D4: LED, Diode_SMD:D_0805_2012Metric, F.Cu at (111.8, 92.1)
- added D5: LED, Diode_SMD:D_0805_2012Metric, F.Cu at (108.7, 92.1)
- added D6: LED, Diode_SMD:D_0805_2012Metric, F.Cu at (105.7, 92.1)
- added D7: WS2812B, LED_SMD:LED_WS2812B_PLCC4_5.0x5.0mm_P3.2mm, F.Cu at (89.2, 102.4)
- added D8: 1N4148W, Diode_SMD:D_SOD-123, F.Cu at (111.3, 104.9)
- added D9: LESD5D5.0CT1G, Diode_SMD:D_SOD-523, F.Cu at (67.4, 109.5)
- added J1: FT232RL, Connector_PinHeader_2.54mm:PinHeader_1x06_P2.54mm_Vertical, F.Cu at (99.1, 116.8)
- added J10: Micro_SD_Card, Library:3M_2908-05WB-MG, F.Cu at (146.5, 77.6)
- added J11: logic_convert, Connector_PinHeader_2.54mm:PinHeader_2x05_P2.54mm_Vertical, F.Cu at (113.9, 83.3)
- added J12: tp, TestPoint:TestPoint_Pad_D1.5mm, B.Cu at (108.7, 132.7)
- added J14: tp, TestPoint:TestPoint_Pad_D1.5mm, B.Cu at (105.1, 129.2)
- added J15: tp, TestPoint:TestPoint_Pad_D1.5mm, B.Cu at (105.1, 132.7)
- added J16: tp, TestPoint:TestPoint_Pad_D1.5mm, B.Cu at (105.1, 136.3)
- added J17: tp, TestPoint:TestPoint_Pad_D1.5mm, B.Cu at (101.6, 129.2)
- added J18: tp, TestPoint:TestPoint_Pad_D1.5mm, B.Cu at (101.6, 132.7)
- added J19: tp, TestPoint:TestPoint_Pad_D1.5mm, B.Cu at (101.6, 136.3)
- added J21: USB_B_Mini, kiC:USB_Mini-B_Lumberg_2486_01_Horizontal, F.Cu at (60.4, 125.0)
- added J22: JTAG, Connector_PinHeader_1.27mm:PinHeader_1x06_P1.27mm_Vertical, F.Cu at (167.5, 119.6)
- added J3: USB_B_Mini, kiC:USB_Mini-B_Lumberg_2486_01_Horizontal, F.Cu at (109.9, 148.4)
- added J5: Oled SSD1306 128x32, Connector_PinHeader_2.54mm:PinHeader_2x03_P2.54mm_Vertical, F.Cu at (122.7, 71.3)
- added J6: FT232RL, Connector_PinHeader_2.54mm:PinHeader_1x06_P2.54mm_Vertical, F.Cu at (99.2, 109.2)
- added J7: ~, Connector_PinHeader_2.54mm:PinHeader_1x07_P2.54mm_Vertical, F.Cu at (134.5, 97.4)
- added J8: tp, TestPoint:TestPoint_Pad_D1.5mm, B.Cu at (108.7, 129.2)
- added J9: Adafruit ST7789, Library:Adafruit_SSD1306_No_Mounting_Holes_pads, F.Cu at (94.6, 58.0)
- added JP10: Jumper_Open, Jumper:SolderJumper-2_P1.3mm_Open_RoundedPad1.0x1.5mm, B.Cu at (108.9, 113.0)
- added JP11: Jumper_Open, Jumper:SolderJumper-2_P1.3mm_Open_RoundedPad1.0x1.5mm, B.Cu at (99.3, 113.0)
- added JP12: Jumper_Open, Jumper:SolderJumper-2_P1.3mm_Open_RoundedPad1.0x1.5mm, B.Cu at (105.7, 113.0)
- added JP13: Jumper_Open, Jumper:SolderJumper-2_P1.3mm_Open_RoundedPad1.0x1.5mm, B.Cu at (102.5, 113.0)
- added JP14: Jumper_Open, Jumper:SolderJumper-2_P1.3mm_Open_RoundedPad1.0x1.5mm, B.Cu at (112.1, 113.0)
- added JP15: Jumper_Open, Jumper:SolderJumper-2_P1.3mm_Open_RoundedPad1.0x1.5mm, B.Cu at (109.8, 122.8)
- added JP16: Jumper_Open, Jumper:SolderJumper-2_P1.3mm_Open_RoundedPad1.0x1.5mm, B.Cu at (113.3, 122.8)
- added JP2: Jumper_2_Open, Jumper:SolderJumper-2_P1.3mm_Open_RoundedPad1.0x1.5mm, B.Cu at (127.3, 110.6)
- added JP3: Jumper_2_Open, Jumper:SolderJumper-2_P1.3mm_Open_RoundedPad1.0x1.5mm, B.Cu at (124.4, 110.5)
- added JP5: NL, Jumper:SolderJumper-2_P1.3mm_Open_RoundedPad1.0x1.5mm, B.Cu at (99.5, 81.1)
- added JP6: NL, Jumper:SolderJumper-2_P1.3mm_Open_RoundedPad1.0x1.5mm, B.Cu at (96.1, 81.1)
- added JP7: 0, Jumper:SolderJumper-2_P1.3mm_Open_RoundedPad1.0x1.5mm, B.Cu at (142.6, 109.9)
- added L1: 100mh, Inductor_SMD:L_1206_3216Metric, F.Cu at (100.4, 142.9)
- added L4: ferrite, Inductor_SMD:L_0805_2012Metric, F.Cu at (143.7, 102.2)
- added L5: ferrite, Inductor_SMD:L_0805_2012Metric, F.Cu at (145.6, 106.0)
- added L6: ferrite, Inductor_SMD:L_0805_2012Metric, F.Cu at (147.8, 110.7)
- added L7: 100mh, Inductor_SMD:L_1206_3216Metric, F.Cu at (74.7, 95.3)
- added LS1: Speaker, Connector_Molex:Molex_Micro-Latch_53253-0270_1x02_P2.00mm_Vertical, F.Cu at (151.1, 108.6)
- added MK1: INMP441ACEZ-R7, kiC:MIC_INMP441ACEZ-R7, F.Cu at (122.5, 104.7)
- added MK2: INMP441ACEZ-R7, kiC:MODULE_OKY3139, F.Cu at (122.2, 104.7)
- added MK3: INMP441ACEZ-R7, kiC:MIC_INMP441ACEZ-R7, B.Cu at (122.5, 104.0)
- added Q10: FDN306P, Package_TO_SOT_SMD:SOT-23W, F.Cu at (95.1, 89.9)
- added Q11: FDN306P, Package_TO_SOT_SMD:SOT-23W, F.Cu at (99.3, 85.6)
- added Q12: 2N7002, Package_TO_SOT_SMD:SOT-23, F.Cu at (107.2, 123.5)
- added Q13: 2N7002, Package_TO_SOT_SMD:SOT-23, F.Cu at (111.7, 123.1)
- added Q14: FDN306P, Package_TO_SOT_SMD:SOT-23W, F.Cu at (118.0, 145.1)
- added Q4: Q_NPN_BCE, Package_TO_SOT_SMD:SOT-23W, F.Cu at (100.7, 104.5)
- added Q5: Q_NPN_BCE, Package_TO_SOT_SMD:SOT-23W, F.Cu at (105.5, 104.5)
- added Q6: 2N7002, Package_TO_SOT_SMD:SOT-23, F.Cu at (90.9, 96.2)
- added Q7: Q_NPN_BCE, Package_TO_SOT_SMD:SOT-23W, F.Cu at (94.3, 78.9)
- added Q8: Q_NPN_BCE, Package_TO_SOT_SMD:SOT-23W, F.Cu at (98.9, 78.9)
- added Q9: 2N7002, Package_TO_SOT_SMD:SOT-23, F.Cu at (99.4, 89.9)
- added R10: 100, Resistor_SMD:R_0805_2012Metric, F.Cu at (100.5, 120.5)
- added R11: 100, Resistor_SMD:R_0805_2012Metric, F.Cu at (101.0, 124.1)
- added R12: 10K, Resistor_SMD:R_0805_2012Metric, F.Cu at (113.2, 135.6)
- added R13: 10K, Resistor_SMD:R_0805_2012Metric, F.Cu at (113.0, 131.9)
- added R14: 1K5, Resistor_SMD:R_0805_2012Metric, F.Cu at (96.6, 140.9)
- added R15: 10k, Resistor_SMD:R_0805_2012Metric, F.Cu at (100.0, 100.4)
- added R16: 10k, Resistor_SMD:R_0805_2012Metric, F.Cu at (108.4, 104.6)
- added R17: 1K5, Resistor_SMD:R_0805_2012Metric, F.Cu at (105.3, 139.2)
- added R18: 10K, Resistor_SMD:R_0805_2012Metric, F.Cu at (94.9, 137.7)
- added R19: 10K, Resistor_SMD:R_0805_2012Metric, F.Cu at (101.1, 140.3)
- added R21: 4K7, Resistor_SMD:R_0805_2012Metric, F.Cu at (98.7, 137.5)
- added R22: 27, Resistor_SMD:R_0805_2012Metric, F.Cu at (109.3, 141.4)
- added R23: 27, Resistor_SMD:R_0805_2012Metric, F.Cu at (105.3, 141.4)
- added R24: 2k2, Resistor_SMD:R_0805_2012Metric, B.Cu at (103.8, 143.1)
- added R25: 1M, Resistor_SMD:R_0805_2012Metric, F.Cu at (138.4, 108.9)
- added R26: 27, Resistor_SMD:R_0805_2012Metric, F.Cu at (70.9, 120.0)
- added R27: 2k2, Resistor_SMD:R_0805_2012Metric, F.Cu at (114.5, 87.7)
- added R28: 2k2, Resistor_SMD:R_0805_2012Metric, F.Cu at (111.6, 87.7)
- added R29: 2k2, Resistor_SMD:R_0805_2012Metric, F.Cu at (108.6, 87.7)
- added R30: 2k2, Resistor_SMD:R_0805_2012Metric, F.Cu at (105.7, 87.7)
- added R31: 2k2, Resistor_SMD:R_0805_2012Metric, F.Cu at (78.3, 134.7)
- added R32: 2k2, Resistor_SMD:R_0805_2012Metric, F.Cu at (61.6, 142.5)
- added R34: 2k2, Resistor_SMD:R_0805_2012Metric, F.Cu at (133.4, 140.3)
- added R36: 2k2, Resistor_SMD:R_0805_2012Metric, F.Cu at (138.5, 137.1)
- added R37: 27, Resistor_SMD:R_0805_2012Metric, F.Cu at (68.8, 120.0)
- added R38: 2k2, Resistor_SMD:R_0805_2012Metric, F.Cu at (87.7, 95.6)
- added R39: 2k2, Resistor_SMD:R_0805_2012Metric, F.Cu at (179.4, 128.4)
- added R41: 2k2, Resistor_SMD:R_0805_2012Metric, F.Cu at (128.1, 76.2)
- added R42: 2k2, Resistor_SMD:R_0805_2012Metric, F.Cu at (125.7, 76.3)
- added R43: 4k7, Resistor_SMD:R_0805_2012Metric, F.Cu at (134.0, 79.8)
- added R44: 4k7, Resistor_SMD:R_0805_2012Metric, F.Cu at (134.0, 73.2)
- added R45: 4k7, Resistor_SMD:R_0805_2012Metric, F.Cu at (134.0, 77.6)
- added R46: 4k7, Resistor_SMD:R_0805_2012Metric, F.Cu at (134.0, 82.0)
- added R47: 4k7, Resistor_SMD:R_0805_2012Metric, F.Cu at (134.0, 75.4)
- added R48: 4k7, Resistor_SMD:R_0805_2012Metric, F.Cu at (147.8, 87.5)
- added R49: 10k, Resistor_SMD:R_0603_1608Metric, F.Cu at (90.6, 79.1)
- added R50: 10k, Resistor_SMD:R_0603_1608Metric, F.Cu at (92.9, 82.5)
- added R51: 10k, Resistor_SMD:R_0603_1608Metric, F.Cu at (96.5, 82.6)
- added R52: 10k, Resistor_SMD:R_0603_1608Metric, F.Cu at (89.9, 76.5)
- added R53: 10k, Resistor_SMD:R_0603_1608Metric, F.Cu at (95.9, 85.5)
- added R54: 2k2, Resistor_SMD:R_0805_2012Metric, F.Cu at (109.4, 119.8)
- added R56: 2k2, Resistor_SMD:R_0805_2012Metric, F.Cu at (116.4, 123.4)
- added R57: 2k2, Resistor_SMD:R_0805_2012Metric, F.Cu at (115.8, 119.9)
- added R58: 5.1k, Resistor_SMD:R_0805_2012Metric, F.Cu at (73.5, 122.7)
- added R59: 5.1k, Resistor_SMD:R_0805_2012Metric, F.Cu at (76.4, 122.7)
- added R6: 10K, Resistor_SMD:R_0805_2012Metric, F.Cu at (113.8, 126.8)
- added R61: 100k, Resistor_SMD:R_0805_2012Metric, F.Cu at (124.1, 116.0)
- added R62: 5.1k, Resistor_SMD:R_0805_2012Metric, F.Cu at (68.3, 114.2)
- added R63: 5.1k, Resistor_SMD:R_0805_2012Metric, F.Cu at (68.3, 111.9)
- added R64: 10K, Resistor_SMD:R_0805_2012Metric, F.Cu at (171.9, 114.5)
- added R65: 100k, Resistor_SMD:R_0805_2012Metric, F.Cu at (179.4, 114.5)
- added R66: 100k, Resistor_SMD:R_0805_2012Metric, F.Cu at (179.4, 117.4)
- added R67: 68k, Resistor_SMD:R_0805_2012Metric, F.Cu at (179.4, 120.4)
- added R7: 10K, Resistor_SMD:R_0603_1608Metric, F.Cu at (113.6, 129.0)
- added SW1: SW_Push, Button_Switch_SMD:SW_Push_SPST_NO_Alps_SKRK, F.Cu at (83.3, 115.5)
- added SW5: left, Button_Switch_SMD:SW_Push_1P1T_NO_CK_KSC9xxG, F.Cu at (137.5, 145.3)
- added SW6: rigth, Button_Switch_SMD:SW_Push_1P1T_NO_CK_KSC9xxG, F.Cu at (75.5, 146.0)
- added SW7: up, Button_Switch_SMD:SW_Push_1P1T_NO_CK_KSC9xxG, F.Cu at (147.4, 136.4)
- added SW8: down, Button_Switch_SMD:SW_Push_1P1T_NO_CK_KSC9xxG, F.Cu at (137.3, 128.0)
- added U1: ESP32-C6-WROOM-1-N8, kiC:XCVR_ESP32-C6-WROOM-1-N8, F.Cu at (71.2, 60.5)
- added U2: ESP32-C6-DEVKITC-1-N8, kiC:MODULE_ESP32-C6-DEVKITC-1-N8, F.Cu at (71.1, 80.0)
- added U3: FT232BM, Package_QFP:LQFP-32_7x7mm_P0.8mm, F.Cu at (104.8, 131.0)
- added U4: LM1117DT-3.3, kiC:SOT-223-3_TabPin2, F.Cu at (95.4, 148.1)
- added U5: MAX98357A, Package_DFN_QFN:TQFN-16-1EP_3x3mm_P0.5mm_EP1.23x1.23mm, F.Cu at (140.4, 105.6)
- added U7: TXS0108EPW, Package_SO:TSSOP-20_4.4x6.5mm_P0.65mm, F.Cu at (108.5, 76.1)
- added U8: 93CxxA, Package_SO:SOIC-8_5.3x5.3mm_P1.27mm, B.Cu at (96.8, 141.5)
- added U9: LM1117DT-3.3, kiC:SOT-223-3_TabPin2, F.Cu at (68.9, 97.7)
- added USBC1: USB3.1C16PFSMT, kiC:USB-C-SMD_TYPE-C-USB-17, F.Cu at (60.0, 112.9)
- added Y2: Crystal, Crystal:Crystal_SMD_EuroQuartz_EQ161-2Pin_3.2x1.5mm, F.Cu at (172.2, 123.1)
Connections:
- D3 pad 1: /IO_0 -> Net-(D3-K)
- D3 pad 2: Net-(D3-A) -> /IO_8
- R33 pad 2: /IO_11 -> BLK_ST7789

Commit message: Update schematics, PCB, and project files
Connections:
- net /EN renamed /esp32_C6/EN
- net /IO_12 renamed /esp32_C6/IO_12
- net /IO_13 renamed /esp32_C6/IO_13
- net /max98357a/GAIN renamed GAIN
- net /max98357a/VCC_MAX98357 renamed VCC_MAX98357
- J7 pad 5: /max98357a/SD -> SD
- MK1 pad 2: /SD -> SD
- MK2 pad 2: /SD -> SD
- MK3 pad 2: /SD -> SD
- R25 pad 2: /max98357a/SD -> SD
- R60 pad 1: /SD -> SD
- R67 pad 1: /max98357a/SD -> SD
- U1 pad 18: /SD -> SD
- U2 pad J3_8: /SD -> SD
Changed lines of the file:
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@@
 			(layers "F.Cu" "F.Mask" "F.Paste")
 			(roundrect_rratio 0.25)
-			(net "/max98357a/VCC_MAX98357")
+			(net "VCC_MAX98357")
 			(pinfunction "1_1")
 			(pintype "passive")
@@
 			(layers "F.Cu" "F.Mask" "F.Paste")
 			(roundrect_rratio 0.243902)
-			(net "/SD")
+			(net "SD")
 			(pintype "passive")
 		)
@@
 			(layers "F.Cu" "F.Mask" "F.Paste")
 			(roundrect_rratio 0.243902)
-			(net "/EN")
+			(net "/esp32_C6/EN")
 			(pintype "passive")
 		)
@@
 			(layers "F.Cu" "F.Mask" "F.Paste")
 			(roundrect_rratio 0.25)
-			(net "/max98357a/VCC_MAX98357")
+			(net "VCC_MAX98357")
 			(pintype "passive")
 		)
@@
 			(layers "*.Cu" "*.Mask")
 			(remove_unused_layers no)
-			(net "/SD")
+			(net "SD")
 			(pinfunction "SD_2")
 			(pintype "output")
@@
 			(layers "F.Cu" "F.Mask" "F.Paste")
 			(roundrect_rratio 0.25)
-			(net "/max98357a/VCC_MAX98357")
+			(net "VCC_MAX98357")
 			(pintype "passive")
 		)
@@
 			(layers "F.Cu" "F.Mask" "F.Paste")
 			(roundrect_rratio 0.25)
-			(net "/EN")
+			(net "/esp32_C6/EN")
 			(pinfunction "2_2")
 			(pintype "passive")
@@
 			(size 1.5 0.9)
 			(layers "F.Cu" "F.Mask" "F.Paste")
-			(net "/EN")
+			(net "/esp32_C6/EN")
 			(pinfunction "EN_3")
 			(pintype "input")
@@
 			(size 1.5 0.9)
 			(layers "F.Cu" "F.Mask" "F.Paste")
-			(net "/IO_12")
+			(net "/esp32_C6/IO_12")
 			(pinfunction "IO12_13")
 			(pintype "bidirectional")
@@
 			(size 1.5 0.9)
 			(layers "F.Cu" "F.Mask" "F.Paste")
-			(net "/IO_13")
+			(net "/esp32_C6/IO_13")
 			(pinfunction "IO13_14")
 			(pintype "bidirectional")
@@
 			(size 1.5 0.9)
 			(layers "F.Cu" "F.Mask" "F.Paste")
-			(net "/SD")
+			(net "SD")
 			(pinfunction "IO20_18")
 			(pintype "bidirectional")
@@
 			(layers "F.Cu" "F.Mask" "F.Paste")
 			(roundrect_rratio 0.243902)
-			(net "/max98357a/VCC_MAX98357")
+			(net "VCC_MAX98357")
 			(pintype "passive")
 		)
@@
 			(layers "F.Cu" "F.Mask" "F.Paste")
 			(roundrect_rratio 0.243902)
-			(net "/max98357a/GAIN")
+			(net "GAIN")
 			(pintype "passive")
 		)
@@
 			(layers "F.Cu" "F.Mask" "F.Paste")
 			(roundrect_rratio 0.243902)
-			(net "/IO_12")
+			(net "/esp32_C6/IO_12")
 			(pintype "passive")
 		)
@@
 			(layers "F.Cu" "F.Mask" "F.Paste")
 			(roundrect_rratio 0.243902)
-			(net "/max98357a/SD")
+			(net "SD")
 			(pintype "passive")
 		)
@@
 			(layers "*.Cu" "*.Mask")
 			(remove_unused_layers no)
-			(net "/max98357a/GAIN")
+			(net "GAIN")
 			(pinfunction "Pin_4_4")
 			(pintype "passive")
@@
 			(layers "*.Cu" "*.Mask")
 			(remove_unused_layers no)
-			(net "/max98357a/SD")
+			(net "SD")
 			(pinfunction "Pin_5_5")
 			(pintype "passive")
@@
 			(layers "*.Cu" "*.Mask")
 			(remove_unused_layers no)
-			(net "/max98357a/VCC_MAX98357")
+			(net "VCC_MAX98357")
 			(pinfunction "Pin_7_7")
 			(pintype "passive")
@@
 			(layers "F.Cu" "F.Mask" "F.Paste")
 			(roundrect_rratio 0.243902)
-			(net "/IO_13")
+			(net "/esp32_C6/IO_13")
 			(pintype "passive")
 		)
@@
 			(layers "F.Cu" "F.Mask" "F.Paste")
 			(roundrect_rratio 0.25)
-			(net "/EN")
+			(net "/esp32_C6/EN")
 			(pintype "passive")
 		)
@@
 			(layers "F.Cu" "F.Mask" "F.Paste")
 			(roundrect_rratio 0.243902)
-			(net "/IO_12")
+			(net "/esp32_C6/IO_12")
 			(pintype "passive")
 		)
@@
 			(layers "F.Cu" "F.Mask" "F.Paste")
 			(roundrect_rratio 0.25)
-			(net "/max98357a/GAIN")
+			(net "GAIN")
 			(pinfunction "GAIN_SLOT_2")
 			(pintype "passive")
@@
 			(layers "F.Cu" "F.Mask" "F.Paste")
 			(roundrect_rratio 0.25)
-			(net "/max98357a/VCC_MAX98357")
+			(net "VCC_MAX98357")
 			(pinfunction "VDD_7")
 			(pintype "power_in")
@@
 			(layers "F.Cu" "F.Mask" "F.Paste")
 			(roundrect_rratio 0.25)
-			(net "/max98357a/VCC_MAX98357")
+			(net "VCC_MAX98357")
 			(pinfunction "VDD_8")
 			(pintype "passive")
@@
 			(layers "F.Cu" "F.Mask" "F.Paste")
 			(roundrect_rratio 0.243902)
-			(net "/max98357a/SD")
+			(net "SD")
 			(pintype "passive")
 		)
@@
 			(layers "F.Cu" "F.Mask" "F.Paste")
 			(roundrect_rratio 0.243902)
-			(net "/IO_13")
+			(net "/esp32_C6/IO_13")
 			(pintype "passive")
 		)
@@
 			(layers "F.Cu" "F.Mask" "F.Paste")
 			(roundrect_rratio 0.25)
-			(net "/EN")
+			(net "/esp32_C6/EN")
 			(pinfunction "C_2")
 			(pintype "passive")
@@
 			(layers "F.Cu" "F.Mask" "F.Paste")
 			(roundrect_rratio 0.25)
-			(net "/max98357a/VCC_MAX98357")
+			(net "VCC_MAX98357")
 			(pinfunction "1_1")
 			(pintype "passive")
@@
 			(layers "F.Cu" "F.Mask" "F.Paste")
 			(roundrect_rratio 0.243902)
-			(net "/max98357a/GAIN")
+			(net "GAIN")
 			(pintype "passive")
 		)
@@
 			(layers "*.Cu" "*.Mask")
 			(remove_unused_layers no)
-			(net "/EN")
+			(net "/esp32_C6/EN")
 			(pinfunction "CHIP_PU_J1_2")
 			(pintype "input")
@@
 			(layers "*.Cu" "*.Mask")
 			(remove_unused_layers no)
-			(net "/SD")
+			(net "SD")
 			(pinfunction "GPIO20_J3_8")
 			(pintype "bidirectional")
@@
 			(layers "*.Cu" "*.Mask")
 			(remove_unused_layers no)
-			(net "/IO_13")
+			(net "/esp32_C6/IO_13")
 			(pinfunction "GPIO13_J3_13")
 			(pintype "bidirectional")
@@
 			(layers "*.Cu" "*.Mask")
 			(remove_unused_layers no)
-			(net "/IO_12")
+			(net "/esp32_C6/IO_12")
 			(pinfunction "GPIO12_J3_14")
 			(pintype "bidirectional")
@@
 			(layers "F.Cu" "F.Mask" "F.Paste")
 			(roundrect_rratio 0.25)
-			(net "/EN")
+			(net "/esp32_C6/EN")
 			(pintype "passive")
 		)
@@
 			(size 0.4 0.6)
 			(layers "F.Cu" "F.Mask")
-			(net "/SD")
+			(net "SD")
 			(pinfunction "SD_2")
 			(pintype "output")
@@
 			(size 0.4 0.6)
 			(layers "B.Cu" "B.Mask")
-			(net "/SD")
+			(net "SD")
 			(pinfunction "SD_2")
 			(pintype "output")

Commit message: Add PWR_FLAG symbols to all schematic sheets to fix power_pin_not_driven ERC errors
Parts:
- moved Y2 113.4 mm to (67.9, 78.6), turned to -90 degrees
- moved R64 111.4 mm to (64.7, 84.5), turned to 180 degrees
- moved C50 108.5 mm to (65.1, 76.3), turned to 90 degrees
- moved C51 107.9 mm to (65.0, 80.7), turned to -90 degrees
- moved J22 99.9 mm to (74.3, 83.7), turned to -90 degrees
- moved D14 91.9 mm to (74.0, 105.9)
- moved C13 89.3 mm to (74.2, 111.7), turned to 180 degrees
- moved C49 78.8 mm to (97.4, 95.3)
- moved R39 73.9 mm to (116.2, 90.2), turned to -90 degrees
- moved D13 70.4 mm to (116.2, 94.6), turned to -90 degrees
- moved R67 46.9 mm to (138.7, 97.1)
- moved R66 43.8 mm to (139.4, 99.7)
- moved R65 33.3 mm to (148.7, 101.7)
- moved D3 2.93 mm to (113.2, 94.5)
- moved D4 2.87 mm to (110.3, 94.5)
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
Commit message: Revert PWR_FLAG additions - remove '??' squares from schematics
Connections:
- J12 pad 1: unconnected-(J12-Pin_1-Pad1) -> /ft232/FT_CTS
- JP15 pad 2: unconnected-(JP15-B-Pad2) -> /ft232/FT_RX
- JP16 pad 2: unconnected-(JP16-B-Pad2) -> /ft232/FT_TX
Changed lines of the file:
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@@
 		(tags "resistor")
 		(property "Reference" "R60"
-			(at 0 -1.65 90)
+			(at 1.778 -2.4892 90)
 			(layer "F.SilkS")
 			(effects
@@
 			(size 1.5 1.5)
 			(layers "B.Cu" "B.Mask")
-			(net "unconnected-(J12-Pin_1-Pad1)")
+			(net "/ft232/FT_CTS")
 			(pinfunction "Pin_1_1")
 			(pintype "passive")
@@
 			(size 1 0.5)
 			(layers "B.Cu" "B.Mask")
-			(net "unconnected-(JP16-B-Pad2)")
+			(net "/ft232/FT_TX")
 			(pinfunction "B_2")
 			(pintype "passive")
@@
 			(size 1 0.5)
 			(layers "B.Cu" "B.Mask")
-			(net "unconnected-(JP15-B-Pad2)")
+			(net "/ft232/FT_RX")
 			(pinfunction "B_2")
 			(pintype "passive")
