File: esp32_xiaozhi.kicad_pcb (KiCad board)
At the start: 4 copper layers, 145.4 x 99.1 mm, 292 parts, among them J1 FT232RL, J10 Micro_SD_Card, J11 tp, J12 tp, J13 tp, J14 Adafruit ST7789, J15 tp, J16 tp, J17 tp, J18 tp, J19 tp, J2 tp_ft232_, J20 tp, J21 USB_B_Mini, J22 Conn_01x05_Pin, J23 TP_VCC, J24 tp, J25 TP_VCC, J26 IDC40, J3 USB_B_Mini, J34 Raspberry_Pi_zero_2w, J4 tp_ft232_, J5 Oled SSD1306 128x32, J53 F32R-1A7H1-11024, J54 tp_epaper, J56 tp_epaper, J57 tp_epaper, J58 tp_epaper, J59 tp_epaper, J6 FT232RL, J8 tp, J9 Adafruit ST7789, Q1 PMOS, Q10 FDN306P, Q11 FDN306P, Q12 FDN306P, Q13 FDN306P, Q14 FDN306P, Q15 2N7002, Q2 BC846, Q3 2N7002, Q4 Q_NPN_BCE, Q5 Q_PNP_BCE, Q6 2N7002, Q7 Q_NPN_BCE, Q8 2N7002, Q9 2N7002, SW1 SW_Push, SW11 boot, SW3 up, SW4 down, SW5 left, SW6 rigth, SW7 Switch_push, SW8 Switch_Push, U1 ESP32-C6-WROOM-1-N8, U10 W25Q128JVSIQ, U11 PIC10F206-IOT, U12 W25Q128JVE, U13 FT232RL, U14 LM1117DT-3.3, U16 TXS0108, U17 TXS0108, U18 TXS0108, U19 M48T08-150PC, U2 ESP32-C6-DEVKITC-1-N8, U3 HS20HS072RX, U4 LM1117DT-3.3, U5 MAX98357A, U6 SS1306_OLEDM0.91_1x-I2C, U8 FT232BM, U9 LM1117DT-3.3, Y2 Oscilador 32768hz, Y3 Crystal_GND24_Small_12MHZ, Y4 Crystal 6MHZ

Commit message: add update
Parts:
- added J27: oled, Connector_PinHeader_2.54mm:PinHeader_1x04_P2.54mm_Vertical, F.Cu at (181.9, 89.5)
- C30: value 100nf -> 1206B104K101NT
- L4: value 10uH @ 305mΩ -> TFM322512ALVA100MTAA
- Y2: value Oscilador 32768hz -> Two pin oscilador 32768hz
- moved C84 1.73 mm to (183.0, 92.7)
Routing:
- net GND: track 678.6 -> 687.7 mm, vias 1109 -> 1117
- net /logic/GPIO3: track 0.00 -> 8.11 mm
- net /logic/GPIO2: track 0.00 -> 5.23 mm
- net +5VC: track 72.7 -> 73.4 mm
