File: esp32_xiaozhi.kicad_sch (KiCad schematic)
At the start: 0 parts

Commit message: ESP32C6 branch changes
Other:
- sheet Battery renamed Clock
- sheet TXS0108E renamed Logic_convert
- removed sheet esp32_s3
- sheet Clock ports: added PCF85263_SCL, PCF85263_SDA; removed none
- sheet display ports: added BLK, CLK, DC, DI, RES, scl, sda; removed none
- sheet esp32_C6 ports: added EN, IO_0, IO_1, IO_10, IO_11, IO_12, IO_13, IO_15, IO_16, IO_17, IO_18, IO_19, IO_2, IO_20, IO_21, IO_22, IO_23, IO_3, IO_4, IO_5, IO_6, IO_7, IO_8, IO_9, MRX, MTX; removed none
- sheet ft232 ports: added mclr; removed none
- sheet led_sw_gpio ports: added led3, led4, led5, led6, sw1, sw2, sw3, sw4, sw5, sw6, sw7, sw8; removed none
- sheet max98357a ports: added BCLK, DIN, GAIN, LRC, SD, pad; removed none

Commit message: Update KiCad project files
Other:
- removed sheet Clock
- added sheet micro_sd (micro_sd.kicad_sch)
- sheet Logic_convert ports: added none; removed B1, B2, B3, B4, B5, B6, B7, B8
- sheet esp32_C6 ports: added RXD0, TXD0; removed IO_16, IO_17
- sheet ft232 ports: added FT_CTS, FT_DTR, FT_RX, FT_TX, FT_VCC, to_CHIP_PU, to_GPIO_0, to_GPIO_EN; removed none
- sheet led_sw_gpio ports: added LED_Data_WS2812; removed none
- sheet max98357a ports: added PAD; removed pad

Commit message: Remove unused schematic files, lock files, and backup directories
Parts:
- added JP10, JP11, JP12, JP13, JP14: Jumper_Open, Jumper:SolderJumper-2_P1.3mm_Open_RoundedPad1.0x1.5mm, symbol Jumper:Jumper_2_Open
Connections:
- net ft232/FT_CTS: now also JP10.1 (A)
- net ft232/FT_DTR: now also JP11.1 (A)
- net ft232/FT_RX: now also JP12.1 (A)
- net ft232/FT_TX: now also JP13.1 (A)
- net ft232/FT_VCC: now also JP14.1 (A)
- new net +3V3: JP14.2 (B)
- new net CTS: JP10.2 (B)
- new net DTR: JP11.2 (B)
- new net MRX: JP13.2 (B)
- new net MTX: JP12.2 (B)
Other:
- sheet esp32_C6 ports: added CTS, DTR; removed MRX, MTX
- sheet ft232 ports: added none; removed to_CHIP_PU, to_GPIO_0, to_GPIO_EN

Commit message: Update all schematic files and project
Other:
- sheet inmp441 ports: added none; removed EN
- sheet led_sw_gpio ports: added WS2812; removed LED_Data_WS2812, sw7, sw8
- note added: "#define BOARD_I2S_BCLK GPIO_NUM_22 // MAX98357A BCLK + INMP441 SCK #define BOARD_I2S_WS GPIO_NUM_23 // MAX98357A LRC + INMP441 WS #define BOARD_I2S_DOUT GPIO_NUM_10 // → MAX98357A DIN #define BOARD_I2S_DIN GPIO_NUM_20 // ← INMP441 SD"
