File: ft232.kicad_sch (KiCad schematic)
At the start: 58 parts, among them J1 FT232RL, J12 tp, J13 tp, J14 tp, J15 tp, J16 tp, J17 tp, J18 tp, J19 tp, J2 tp_ft232_, J20 tp, J3 USB_B_Mini, J4 tp_ft232_, J8 tp, Q12 2N7002, Q13 2N7002, Q14 FDN306P, U3 FT232BM, U4 LM1117DT-3.3, U8 93CxxA, Y1 Crystal

Commit message: Update schematics, PCB, and project files
Connections:
- net FT_CTS: now also J12.1 (Pin_1)
- net FT_RX: now also JP15.2 (B)
- net FT_TX: now also JP16.2 (B)
Changed lines of the file:
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@@
 	)
 	(junction
+		(at 204.47 85.09)
+		(diameter 0)
+		(color 0 0 0 0)
+	)
+	(junction
 		(at 115.57 201.93)
 		(diameter 0)
@@
 	)
 	(junction
+		(at 212.09 96.52)
+		(diameter 0)
+		(color 0 0 0 0)
+	)
+	(junction
 		(at 359.41 49.53)
 		(diameter 0)
@@
 	)
 	(junction
-		(at 289.56 77.47)
-		(diameter 0)
-		(color 0 0 0 0)
-	)
-	(junction
 		(at 101.6 209.55)
 		(diameter 0)
@@
 	)
 	(junction
-		(at 212.09 99.06)
-		(diameter 0)
-		(color 0 0 0 0)
-	)
-	(junction
 		(at 168.91 168.91)
 		(diameter 0)
@@
 	)
 	(junction
-		(at 207.01 82.55)
-		(diameter 0)
-		(color 0 0 0 0)
-	)
-	(junction
 		(at 148.59 83.82)
 		(diameter 0)
@@
 	(wire
 		(pts
+			(xy 207.01 97.79) (xy 207.01 99.06)
+		)
+		(stroke
+			(width 0)
+			(type default)
+		)
+	)
+	(wire
+		(pts
 			(xy 231.14 200.66) (xy 238.76 200.66)
 		)
@@
 	(wire
 		(pts
-			(xy 212.09 93.98) (xy 212.09 99.06)
+			(xy 212.09 93.98) (xy 212.09 96.52)
 		)
 		(stroke
@@
 	(wire
 		(pts
-			(xy 287.02 77.47) (xy 287.02 73.66)
-		)
-		(stroke
-			(width 0)
-			(type default)
-		)
-	)
-	(wire
-		(pts
-			(xy 101.6 214.63) (xy 101.6 209.55)
+			(xy 287.02 80.01) (xy 287.02 73.66)
 		)
 		(stroke
@@
 	(wire
 		(pts
-			(xy 287.02 77.47) (xy 289.56 77.47)
+			(xy 182.88 158.75) (xy 182.88 152.4)
 		)
 		(stroke
@@
 	(wire
 		(pts
-			(xy 182.88 158.75) (xy 182.88 152.4)
+			(xy 302.26 68.58) (xy 297.18 68.58)
 		)
 		(stroke
@@
 	(wire
 		(pts
-			(xy 302.26 68.58) (xy 297.18 68.58)
+			(xy 359.41 49.53) (xy 353.06 49.53)
 		)
 		(stroke
@@
 	(wire
 		(pts
-			(xy 359.41 49.53) (xy 353.06 49.53)
+			(xy 218.44 96.52) (xy 212.09 96.52)
 		)
 		(stroke
@@
 	(wire
 		(pts
-			(xy 218.44 99.06) (xy 212.09 99.06)
+			(xy 110.49 140.97) (xy 109.22 140.97)
 		)
 		(stroke
@@
 	(wire
 		(pts
-			(xy 110.49 140.97) (xy 109.22 140.97)
+			(xy 208.28 85.09) (xy 208.28 97.79)
 		)
 		(stroke
@@
 	(wire
 		(pts
-			(xy 207.01 82.55) (xy 209.55 82.55)
+			(xy 204.47 82.55) (xy 209.55 82.55)
+		)
+		(stroke
+			(width 0)
+			(type default)
+		)
+	)
+	(wire
+		(pts
+			(xy 208.28 97.79) (xy 207.01 97.79)
 		)
 		(stroke
@@
 	(wire
 		(pts
+			(xy 101.6 214.63) (xy 101.6 209.55)
+		)
+		(stroke
+			(width 0)
+			(type default)
+		)
+	)
+	(wire
+		(pts
 			(xy 332.74 49.53) (xy 332.74 50.8)
 		)
@@
 	(wire
 		(pts
+			(xy 218.44 96.52) (xy 218.44 99.06)
+		)
+		(stroke
+			(width 0)
+			(type default)
+		)
+	)
+	(wire
+		(pts
 			(xy 322.58 66.04) (xy 322.58 68.58)
 		)
@@
 	(wire
 		(pts
-			(xy 44.45 157.48) (xy 33.02 157.48)
+			(xy 212.09 96.52) (xy 212.09 99.06)
 		)
 		(stroke
@@
 	(wire
 		(pts
-			(xy 207.01 82.55) (xy 207.01 99.06)
+			(xy 44.45 157.48) (xy 33.02 157.48)
 		)
 		(stroke
@@
 	(wire
 		(pts
+			(xy 147.32 59.69) (xy 140.97 59.69)
+		)
+		(stroke
+			(width 0)
+			(type default)
+		)
+	)
+	(wire
+		(pts
 			(xy 172.72 157.48) (xy 172.72 158.75)
 		)
@@
 	(wire
 		(pts
-			(xy 204.47 82.55) (xy 204.47 99.06)
+			(xy 204.47 82.55) (xy 204.47 85.09)
 		)
 		(stroke
@@
 	(wire
 		(pts
-			(xy 204.47 82.55) (xy 207.01 82.55)
+			(xy 204.47 85.09) (xy 204.47 99.06)
 		)
 		(stroke
@@
 	(wire
 		(pts
+			(xy 97.79 214.63) (xy 101.6 214.63)
+		)
+		(stroke
+			(width 0)
+			(type default)
+		)
+	)
+	(wire
+		(pts
 			(xy 140.97 71.12) (xy 135.89 71.12)
 		)
@@
 	(wire
 		(pts
+			(xy 208.28 85.09) (xy 204.47 85.09)
+		)
+		(stroke
+			(width 0)
+			(type default)
+		)
+	)
+	(wire
+		(pts
 			(xy 184.15 142.24) (xy 165.1 142.24)
 		)
@@
 		)
 	)
+	(wire
+		(pts
+			(xy 147.32 50.8) (xy 140.97 50.8)
+		)
+		(stroke
+			(width 0)
+			(type default)
+		)
+	)
 	(label "FT_RX"
 		(at 157.48 109.22 180)
@@
 		)
 	)
+	(label "FT_RX"
+		(at 147.32 59.69 0)
+		(effects
+			(font
+				(size 1.27 1.27)
+			)
+			(justify left bottom)
+		)
+	)
 	(label "TX"
 		(at 123.19 50.8 0)
@@
 		)
 	)
+	(label "FT_TX"
+		(at 147.32 50.8 0)
+		(effects
+			(font
+				(size 1.27 1.27)
+			)
+			(justify left bottom)
+		)
+	)
 	(label "FT_USB_BM"
 		(at 323.85 68.58 0)
@@
 	(symbol
 		(lib_id "Connector:Conn_01x01_Pin")
-		(at 28.1354 154.5821 0)
+		(at 27.94 154.94 0)
 		(unit 1)
 		(body_style 1)
@@
 		(dnp no)
 		(property "Reference" "J12"
-			(at 26.6114 153.3121 0)
+			(at 26.416 153.67 0)
 			(show_name no)
 			(do_not_autoplace no)
@@
 		)
 		(property "Value" "tp"
-			(at 34.9934 153.3121 0)
+			(at 34.798 153.67 0)
 			(show_name no)
 			(do_not_autoplace no)
@@
 		)
 		(property "Footprint" "TestPoint:TestPoint_Pad_D1.5mm"
-			(at 28.1354 154.5821 0)
+			(at 27.94 154.94 0)
 			(hide yes)
 			(show_name no)
@@
 		)
 		(property "Datasheet" ""
-			(at 28.1354 154.5821 0)
+			(at 27.94 154.94 0)
 			(hide yes)
 			(show_name no)
@@
 		)
 		(property "Description" "Generic connector, single row, 01x01, script generated"
-			(at 28.1354 154.5821 0)
+			(at 27.94 154.94 0)
 			(hide yes)
 			(show_name no)
@@
 	)
 	(symbol
+		(lib_id "power:GND1")
+		(at 287.02 80.01 0)
+		(unit 1)
+		(body_style 1)
+		(exclude_from_sim no)
+		(in_bom yes)
+		(on_board yes)
+		(in_pos_files yes)
+		(dnp no)
+		(fields_autoplaced yes)
+		(property "Reference" "#PWR0141"
+			(at 287.02 86.36 0)
+			(hide yes)
+			(show_name no)
+			(do_not_autoplace no)
+			(effects
+				(font
+					(size 1.27 1.27)
+				)
+			)
+		)
+		(property "Value" "GND"
+			(at 287.02 85.09 0)
+			(show_name no)
+			(do_not_autoplace no)
+			(effects
+				(font
+					(size 1.27 1.27)
+				)
+			)
+		)
+		(property "Footprint" ""
+			(at 287.02 80.01 0)
+			(hide yes)
+			(show_name no)
+			(do_not_autoplace no)
+			(effects
+				(font
+					(size 1.27 1.27)
+				)
+			)
+		)
+		(property "Datasheet" ""
+			(at 287.02 80.01 0)
+			(hide yes)
+			(show_name no)
+			(do_not_autoplace no)
+			(effects
+				(font
+					(size 1.27 1.27)
+				)
+			)
+		)
+		(property "Description" ""
+			(at 287.02 80.01 0)
+			(show_name no)
+			(do_not_autoplace no)
+			(effects
+				(font
+					(size 1.27 1.27)
+				)
+			)
+		)
+		(pin "1"
+		)
+		(instances
+			(project "esp32_xiaozhi"
+				(path "/cae338e8-f342-43cb-b99a-a0486629133c/62520ce4-d21b-4842-a32d-5b11b343b2aa"
+					(reference "#PWR0141")
+					(unit 1)
+				)
+			)
+		)
+	)
+	(symbol
 		(lib_id "Device:R")
 		(at 172.72 162.56 180)
@@
 	(symbol
 		(lib_id "power:GND1")
-		(at 101.6 214.63 0)
+		(at 97.79 214.63 0)
 		(unit 1)
 		(body_style 1)
@@
 		(fields_autoplaced yes)
 		(property "Reference" "#PWR014"
-			(at 101.6 220.98 0)
+			(at 97.79 220.98 0)
 			(hide yes)
 			(show_name no)
@@
 		)
 		(property "Value" "GND1"
-			(at 101.6 219.71 0)
+			(at 97.79 219.71 0)
 			(show_name no)
 			(do_not_autoplace no)
@@
 		)
 		(property "Footprint" ""
-			(at 101.6 214.63 0)
+			(at 97.79 214.63 0)
 			(hide yes)
 			(show_name no)
@@
 		)
 		(property "Datasheet" ""
-			(at 101.6 214.63 0)
+			(at 97.79 214.63 0)
 			(hide yes)
 			(show_name no)
@@
 		)
 		(property "Description" ""
-			(at 101.6 214.63 0)
+			(at 97.79 214.63 0)
 			(show_name no)
 			(do_not_autoplace no)
