File: ft232.kicad_sch (KiCad schematic)
At the start: 51 parts, among them J1 FT232RL, J12 tp, J13 tp, J15 tp, J16 tp, J17 tp, J19 tp, J2 tp_ft232_, J20 tp, J24 tp, J3 USB_B_Mini, J4 tp_ft232_, J8 tp, Q14 FDN306P, U13 FT232RL, U4 LM1117DT-3.3, Y3 Crystal_GND24_Small_6MHZ

Commit message: Actualización de esquemas, PCB y librerías
Parts:
- C17, C4, C47, C5, C54, C6, C7, C9: LCSC C1525 -> C28233
- C18: value 100nf -> 4.7uf; LCSC C1525 -> C1779
- C48: LCSC C28323 -> C1779
- C57: value 1uf -> 4.7uf; LCSC C28323 -> C1779
- D1, D6: value RX -> RX led Green
- D2: value RX -> RX white / Yellow
- R10, R11: value 100 -> 0
Changed lines of the file:
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@@
 			)
 		)
-		(property "LCSC" "C1525"
+		(property "LCSC" "C28233"
 			(at 66.04 254 0)
 			(hide yes)
@@
 			)
 		)
-		(property "Value" "1uf"
+		(property "Value" "4.7uf"
 			(at 269.494 156.464 90)
 			(show_name no)
@@
 			)
 		)
-		(property "LCSC" "C28323  "
+		(property "LCSC" "C1779"
 			(at 266.7 163.83 90)
 			(hide yes)
@@
 			)
 		)
-		(property "LCSC" "C1525"
+		(property "LCSC" "C28233"
 			(at 335.28 177.8 90)
 			(hide yes)
@@
 			)
 		)
-		(property "LCSC" "C1525"
+		(property "LCSC" "C28233"
 			(at 351.79 41.91 0)
 			(hide yes)
@@
 			)
 		)
-		(property "Value" "RX"
-			(at 240.03 227.3935 90)
+		(property "Value" "RX white / Yellow"
+			(at 248.666 227.584 90)
 			(show_name no)
 			(do_not_autoplace no)
@@
 		)
 		(property "Description" "Light emitting diode Blue"
-			(at 244.856 227.33 0)
+			(at 236.22 212.09 0)
 			(show_name no)
 			(do_not_autoplace no)
@@
 			)
 		)
-		(property "LCSC" "C1525"
+		(property "LCSC" "C28233"
 			(at 335.28 185.42 90)
 			(hide yes)
@@
 			)
 		)
-		(property "LCSC" "C1525"
+		(property "LCSC" "C28233"
 			(at 78.74 254 0)
 			(hide yes)
@@
 			)
 		)
-		(property "LCSC" "C1525"
+		(property "LCSC" "C28233"
 			(at 245.11 176.53 90)
 			(hide yes)
@@
 			)
 		)
-		(property "Value" "100"
+		(property "Value" "0"
 			(at 249.428 94.234 90)
 			(show_name no)
@@
 			)
 		)
-		(property "LCSC" "C1525"
+		(property "LCSC" "C28233"
 			(at 105.41 254 0)
 			(hide yes)
@@
 			)
 		)
-		(property "Value" "RX"
+		(property "Value" "RX led Green"
 			(at 274.32 170.1165 90)
 			(show_name no)
@@
 			)
 		)
-		(property "Value" "100"
+		(property "Value" "0"
 			(at 249.428 88.392 90)
 			(show_name no)
@@
 			)
 		)
-		(property "Value" "100nf"
+		(property "Value" "4.7uf"
 			(at 385.318 39.878 0)
 			(show_name no)
@@
 			)
 		)
-		(property "LCSC" "C1525"
+		(property "LCSC" "C1779"
 			(at 378.46 41.91 0)
 			(hide yes)
@@
 			)
 		)
-		(property "LCSC" "C1525"
+		(property "LCSC" "C28233"
 			(at 92.71 254 0)
 			(hide yes)
@@
 			)
 		)
-		(property "LCSC" "C28323  "
+		(property "LCSC" "C1779"
 			(at 250.19 187.96 90)
 			(hide yes)
@@
 			)
 		)
-		(property "Value" "RX"
-			(at 232.41 227.3935 90)
+		(property "Value" "RX led Green"
+			(at 213.868 228.346 90)
 			(show_name no)
 			(do_not_autoplace no)

Commit message: update files
Parts:
- U13: LCSC C49018905 -> C8690
- Y3: value Crystal_GND24_Small_6MHZ -> Crystal_GND24_Small_12MHZ
Changed lines of the file:
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@@
 			)
 		)
-		(property "Value" "Crystal_GND24_Small_6MHZ"
+		(property "Value" "Crystal_GND24_Small_12MHZ"
 			(at 334.01 211.328 0)
 			(show_name no)
@@
 			)
 		)
-		(property "LCSC" "C49018905"
+		(property "LCSC" "C8690"
 			(at 181.61 107.95 0)
 			(hide yes)
