File: inmp441.kicad_sch (KiCad schematic)
At the start: 0 parts

Commit message: Add components: TXS0108E, FT232 oscillators/power/USB, symbol library table
Parts:
- added MK1: INMP441ACEZ-R7, kiC:MIC_INMP441ACEZ-R7, symbol INMP441ACEZ-R7:INMP441ACEZ-R7
Connections:
- new net GND: MK1.5 (GND), MK1.6 (GND), MK1.9 (GND)
Changed lines of the file:
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@@
 	(generator_version "10.0")
 	(paper "A4")
+	(symbol
+		(lib_id "INMP441ACEZ-R7:INMP441ACEZ-R7")
+		(at 139.7 92.71 0)
+		(unit 1)
+		(body_style 1)
+		(exclude_from_sim no)
+		(in_bom yes)
+		(on_board yes)
+		(in_pos_files yes)
+		(dnp no)
+		(fields_autoplaced yes)
+		(property "Reference" "MK1"
+			(at 139.7 77.47 0)
+			(show_name no)
+			(do_not_autoplace no)
+			(effects
+				(font
+					(size 1.27 1.27)
+				)
+			)
+		)
+		(property "Value" "INMP441ACEZ-R7"
+			(at 139.7 80.01 0)
+			(show_name no)
+			(do_not_autoplace no)
+			(effects
+				(font
+					(size 1.27 1.27)
+				)
+			)
+		)
+		(property "Footprint" "kiC:MIC_INMP441ACEZ-R7"
+			(at 139.7 92.71 0)
+			(hide yes)
+			(show_name no)
+			(do_not_autoplace no)
+			(effects
+				(font
+					(size 1.27 1.27)
+				)
+				(justify bottom)
+			)
+		)
+		(property "Datasheet" ""
+			(at 139.7 92.71 0)
+			(hide yes)
+			(show_name no)
+			(do_not_autoplace no)
+			(effects
+				(font
+					(size 1.27 1.27)
+				)
+			)
+		)
+		(property "Description" "60 Hz ~ 15 kHz Digital, I2S Microphone MEMS (Silicon) 1.62 V ~ 3.63 V Omnidirectional (-26dB ±3dB @ 94dB SPL) Solder Pads"
+			(at 139.7 92.71 0)
+			(hide yes)
+			(show_name no)
+			(do_not_autoplace no)
+			(effects
+				(font
+					(size 1.27 1.27)
+				)
+				(justify bottom)
+			)
+		)
+		(property "MF" "TDK InvenSense"
+			(at 139.7 92.71 0)
+			(hide yes)
+			(show_name no)
+			(do_not_autoplace no)
+			(effects
+				(font
+					(size 1.27 1.27)
+				)
+				(justify bottom)
+			)
+		)
+		(property "MAXIMUM_PACKAGE_HEIGHT" "1.05 mm"
+			(at 139.7 92.71 0)
+			(hide yes)
+			(show_name no)
+			(do_not_autoplace no)
+			(effects
+				(font
+					(size 1.27 1.27)
+				)
+				(justify bottom)
+			)
+		)
+		(property "Package" "LGA-9 TDK InvenSense"
+			(at 139.7 92.71 0)
+			(hide yes)
+			(show_name no)
+			(do_not_autoplace no)
+			(effects
+				(font
+					(size 1.27 1.27)
+				)
+				(justify bottom)
+			)
+		)
+		(property "Price" "None"
+			(at 139.7 92.71 0)
+			(hide yes)
+			(show_name no)
+			(do_not_autoplace no)
+			(effects
+				(font
+					(size 1.27 1.27)
+				)
+				(justify bottom)
+			)
+		)
+		(property "Check_prices" "https://www.snapeda.com/parts/INMP441ACEZ-R7/TDK/view-part/?ref=eda"
+			(at 139.7 92.71 0)
+			(hide yes)
+			(show_name no)
+			(do_not_autoplace no)
+			(effects
+				(font
+					(size 1.27 1.27)
+				)
+				(justify bottom)
+			)
+		)
+		(property "STANDARD" "Manufacturer Recommendations"
+			(at 139.7 92.71 0)
+			(hide yes)
+			(show_name no)
+			(do_not_autoplace no)
+			(effects
+				(font
+					(size 1.27 1.27)
+				)
+				(justify bottom)
+			)
+		)
+		(property "PARTREV" "1.1"
+			(at 139.7 92.71 0)
+			(hide yes)
+			(show_name no)
+			(do_not_autoplace no)
+			(effects
+				(font
+					(size 1.27 1.27)
+				)
+				(justify bottom)
+			)
+		)
+		(property "SnapEDA_Link" "https://www.snapeda.com/parts/INMP441ACEZ-R7/TDK/view-part/?ref=snap"
+			(at 139.7 92.71 0)
+			(hide yes)
+			(show_name no)
+			(do_not_autoplace no)
+			(effects
+				(font
+					(size 1.27 1.27)
+				)
+				(justify bottom)
+			)
+		)
+		(property "MP" "INMP441ACEZ-R7"
+			(at 139.7 92.71 0)
+			(hide yes)
+			(show_name no)
+			(do_not_autoplace no)
+			(effects
+				(font
+					(size 1.27 1.27)
+				)
+				(justify bottom)
+			)
+		)
+		(property "Purchase-URL" "https://www.snapeda.com/api/url_track_click_mouser/?unipart_id=76082&manufacturer=TDK InvenSense&part_name=INMP441ACEZ-R7&search_term=inmp441"
+			(at 139.7 92.71 0)
+			(hide yes)
+			(show_name no)
+			(do_not_autoplace no)
+			(effects
+				(font
+					(size 1.27 1.27)
+				)
+				(justify bottom)
+			)
+		)
+		(property "Availability" "In Stock"
+			(at 139.7 92.71 0)
+			(hide yes)
+			(show_name no)
+			(do_not_autoplace no)
+			(effects
+				(font
+					(size 1.27 1.27)
+				)
+				(justify bottom)
+			)
+		)
+		(property "MANUFACTURER" "TDK InvenSense"
+			(at 139.7 92.71 0)
+			(hide yes)
+			(show_name no)
+			(do_not_autoplace no)
+			(effects
+				(font
+					(size 1.27 1.27)
+				)
+				(justify bottom)
+			)
+		)
+		(pin "1"
+		)
+		(pin "9"
+		)
+		(pin "8"
+		)
+		(pin "5"
+		)
+		(pin "6"
+		)
+		(pin "7"
+		)
+		(pin "3"
+		)
+		(pin "4"
+		)
+		(pin "2"
+		)
+		(instances
+			(project "esp32_xiaozhi"
+				(path "/cae338e8-f342-43cb-b99a-a0486629133c/d2e61921-5974-44e2-9221-de7c05f17e70"
+					(reference "MK1")
+					(unit 1)
+				)
+			)
+		)
+	)
 )

Commit message: ESP32S3 branch initial changes
Parts:
- added C27: 100nf, Capacitor_SMD:C_0805_2012Metric, symbol Device:C
- added L6, L7: ferrite, Inductor_SMD:L_0805_2012Metric, symbol Device:L
- added R38: 1M, Resistor_SMD:R_0805_2012Metric, symbol Device:R
Connections:
- net GND: now also C27.1, R38.2
- net SCK: now reaches MK1.1 (SCK)
- net SD: now reaches MK1.2 (SD)
- net WS: now reaches MK1.3 (WS)
- net L/R: now reaches MK1.4 (L/R)
- net L/R: now also R38.1
- net at MK1.7 (VDD): now also C27.2, L6.1, L7.1
- net EN: now reaches MK1.8 (CHIPEN)
- new net +3V3: L6.2
- new net +5V: L7.2

Commit message: Update KiCad project files
Parts:
- removed L6: ferrite, Inductor_SMD:L_0805_2012Metric, symbol Device:L
- added J5, J6: Conn_01x03_Pin, Connector_PinHeader_2.54mm:PinHeader_1x03_P2.54mm_Vertical, symbol Connector:Conn_01x03_Pin
- added JP2: Jumper_2_Open, Jumper:SolderJumper-2_P1.3mm_Bridged_RoundedPad1.0x1.5mm, symbol Jumper:Jumper_2_Open
- added JP3, JP4: Jumper_2_Open, Jumper:SolderJumper-2_P1.3mm_Open_RoundedPad1.0x1.5mm, symbol Jumper:Jumper_2_Open
- renumbered C27 to C19, L7 to L2, R38 to R24
Connections:
- net +3V3: now also JP4.2 (B)
- net +5V: now also JP3.2 (B); no longer L2.2
- net EN: now also J5.2 (Pin_2)
- net GND: now also J6.1 (Pin_1), JP2.1 (A)
- net L/R: now also J5.3 (Pin_3), JP2.2 (B)
- net SCK: now also J5.1 (Pin_1)
- net WS: now also J6.2 (Pin_2)
- net at C19.2, L2.1, MK1.7 (VDD): now also J6.3 (Pin_3)
- new net: JP3.1 (A), JP4.1 (A), L2.2
Other:
- moved on the sheet: C19, L2, R24

Commit message: Remove unused schematic files, lock files, and backup directories
Parts:
- removed J5, J6: Conn_01x03_Pin, Connector_PinHeader_2.54mm:PinHeader_1x03_P2.54mm_Vertical, symbol Connector:Conn_01x03_Pin
- removed R24: 1M, Resistor_SMD:R_0805_2012Metric, symbol Device:R
- added MK2: INMP441ACEZ-R7, kiC:MODULE_OKY3139, symbol INMP441ACEZ-R7:INMP441ACEZ-R7
- JP2: footprint Jumper:SolderJumper-2_P1.3mm_Bridged_RoundedPad1.0x1.5mm -> Jumper:SolderJumper-2_P1.3mm_Open_RoundedPad1.0x1.5mm
- JP3, JP4: value Jumper_2_Open -> Jumper_Open
Connections:
- net EN: now also MK2.8 (CHIPEN)
- net GND: now also MK2.5 (GND), MK2.6 (GND), MK2.9 (GND)
- net L/R: now also MK2.4 (L/R)
- net SCK: now also MK2.1 (SCK)
- net SD: now also MK2.2 (SD)
- net WS: now also MK2.3 (WS)
- net VDD_INMP441: now reaches C19.2, L2.1, MK1.7 (VDD)
- net VDD_INMP441: now also MK2.7 (VDD)

Commit message: Update all schematic files and project
Parts:
- removed JP4: Jumper_Open, Jumper:SolderJumper-2_P1.3mm_Open_RoundedPad1.0x1.5mm, symbol Jumper:Jumper_2_Open
- added MK3: INMP441ACEZ-R7, kiC:MIC_INMP441ACEZ-R7, symbol INMP441ACEZ-R7:INMP441ACEZ-R7
- added R60, R61: 100k, Resistor_SMD:R_0805_2012Metric, symbol Device:R
- JP3: value Jumper_Open -> Jumper_2_Open
Connections:
- net +5V is gone; now on net +3V3: JP3.2 (B)
- net VDD_INMP441 is gone; now on net EN: C19.2, L2.1, MK1.7 (VDD), MK2.7 (VDD)
- net +3V3: now also L2.2
- net EN: now also MK3.7 (VDD), MK3.8 (CHIPEN)
- net GND: now also MK3.5 (GND), MK3.6 (GND), MK3.9 (GND), R60.2, R61.2
- net L/R: now also JP3.1 (A), MK3.4 (L/R), R61.1
- net SCK: now also MK3.1 (SCK)
- net SD: now also MK3.2 (SD), R60.1
- net WS: now also MK3.3 (WS)
Other:
- moved on the sheet: C19, JP2, L2, MK1

Commit message: Update all schematic files and project
Other:
- moved on the sheet: C19, JP2, JP3, L2, MK1, MK2, MK3, R60, R61

Commit message: Update schematics, PCB, and project files
Other:
- moved on the sheet: MK1

Commit message: Add PWR_FLAG symbols to all schematic sheets to fix power_pin_not_driven ERC errors
Changed lines of the file:
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@@
+		)
+	)
+	(symbol
+		(lib_id "power:PWR_FLAG")
+		(at 50.0 50.0 0)
+		(unit 1)
+		(body_style 1)
+		(exclude_from_sim no)
+		(in_bom no)
+		(on_board yes)
+		(in_pos_files no)
+		(dnp no)
+		(property "Reference" "#FLG040"
+			(at 50.0 45.0 0)
+			(hide yes)
+			(show_name no)
+			(do_not_autoplace no)
+			(effects
+				(font
+					(size 1.27 1.27)
+				)
+			)
+		)
+		(property "Value" "PWR_FLAG"
+			(at 50.0 55.0 0)
+			(hide yes)
+			(show_name no)
+			(do_not_autoplace no)
+			(effects
+				(font
+					(size 1.27 1.27)
+				)
+			)
+		)
+		(pin "1"
+			(uuid "e3f4a5b6-7890-12cd-ef01-234567890123-pin1")
+		)
+		(instances
+			(project "esp32_xiaozhi"
+				(path "/cae338e8-f342-43cb-b99a-a0486629133c/d2e61921-5974-44e2-9221-de7c05f17e70"
+					(reference "#FLG040")
+					(unit 1)
+				)
+			)
+		)
+	)
+	(symbol
+		(lib_id "power:PWR_FLAG")
+		(at 50.0 100.0 0)
+		(unit 1)
+		(body_style 1)
+		(exclude_from_sim no)
+		(in_bom no)
+		(on_board yes)
+		(in_pos_files no)
+		(dnp no)
+		(property "Reference" "#FLG041"
+			(at 50.0 95.0 0)
+			(hide yes)
+			(show_name no)
+			(do_not_autoplace no)
+			(effects
+				(font
+					(size 1.27 1.27)
+				)
+			)
+		)
+		(property "Value" "PWR_FLAG"
+			(at 50.0 105.0 0)
+			(hide yes)
+			(show_name no)
+			(do_not_autoplace no)
+			(effects
+				(font
+					(size 1.27 1.27)
+				)
+			)
+		)
+		(pin "1"
+			(uuid "e3f4a5b6-7890-12cd-ef01-234567890124-pin1")
+		)
+		(instances
+			(project "esp32_xiaozhi"
+				(path "/cae338e8-f342-43cb-b99a-a0486629133c/d2e61921-5974-44e2-9221-de7c05f17e70"
+					(reference "#FLG041")
+					(unit 1)
+				)
+			)
 		)
 	)
