File: display.kicad_sch (KiCad schematic)
At the start: 0 parts

Commit message: Add components: TXS0108E, FT232 oscillators/power/USB, symbol library table
Parts:
- added J21: conector oled ST1306 128x32, Connector_PinHeader_2.54mm:PinHeader_2x03_P2.54mm_Vertical, symbol Connector_Generic:Conn_01x06
- added J22: Adafruit ST7789, Library:Adafruit_SSD1306_No_Mounting_Holes_pads, symbol Connector:Conn_01x07_Pin
- added R31, R32: 1k, Resistor_SMD:R_0805_2012Metric, symbol Device:R
Connections:
- new net +3.3V: J21.2 (Pin_2), J22.2 (Pin_2), R31.1, R32.1
- new net GND: J21.1 (Pin_1), J22.1 (Pin_1)
- new net RG0: J22.5 (Pin_5)
- new net RG1: J22.6 (Pin_6)
- new net RG6: J22.7 (Pin_7)
- new net RG7: J21.4 (Pin_4)
- new net RG8: J21.6 (Pin_6)
- new net scl: J21.5 (Pin_5), J22.4 (Pin_4), R31.2
- new net sda: J21.3 (Pin_3), J22.3 (Pin_3), R32.2

Commit message: ESP32S3 branch initial changes
Parts:
- added U7: ER_OLEDM0.91_1x-I2C, Connector_PinHeader_2.54mm:PinHeader_1x04_P2.54mm_Vertical, symbol Display_Graphic:ER_OLEDM0.91_1x-I2C
- J21: value conector oled ST1306 128x32 -> Oled SSD1306 128x32
- R31, R32: value 1k -> 2k2
Connections:
- net RG8 is gone; now on net GND: J21.6 (Pin_6)
- net +3.3V: now also J21.1 (Pin_1), U7.2 (VCC); no longer J21.2 (Pin_2), R31.1, R32.1
- net GND: now also U7.1 (GND); no longer J21.1 (Pin_1)
- net scl: now also U7.3 (SCL); no longer J22.4 (Pin_4)
- net sda: now also U7.4 (SDA); no longer J22.3 (Pin_3)
- net RG0 renamed RES
- net RG1 renamed DC
- net RG6 renamed BLK
- net RG7 renamed +5V
- net +5V: now also J21.2 (Pin_2)
- new net +3V3: R31.1, R32.1
- new net CLK: J22.4 (Pin_4)
- new net DI: J22.3 (Pin_3)

Commit message: ESP32C6 branch changes
Other:
- moved on the sheet: U7
Changed lines of the file:
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@@
 	)
 	(label "SCL"
-		(at 41.91 74.93 180)
+		(at 80.01 80.01 180)
 		(effects
 			(font
@@
 	)
 	(label "SDA"
-		(at 41.91 80.01 180)
+		(at 80.01 85.09 180)
 		(effects
 			(font
@@
 	(symbol
 		(lib_id "power:+3.3V")
-		(at 52.07 67.31 0)
+		(at 90.17 72.39 0)
 		(unit 1)
 		(body_style 1)
@@
 		(fields_autoplaced yes)
 		(property "Reference" "#PWR069"
-			(at 52.07 71.12 0)
+			(at 90.17 76.2 0)
 			(hide yes)
 			(show_name no)
@@
 		)
 		(property "Value" "+3.3V"
-			(at 52.07 62.23 0)
+			(at 90.17 67.31 0)
 			(show_name no)
 			(do_not_autoplace no)
@@
 		)
 		(property "Footprint" ""
-			(at 52.07 67.31 0)
-			(hide yes)
-			(show_name no)
-			(do_not_autoplace no)
-			(effects
-				(font
-					(size 1.27 1.27)
-				)
-			)
-		)
-		(property "Datasheet" ""
-			(at 52.07 67.31 0)
+			(at 90.17 72.39 0)
+			(hide yes)
+			(show_name no)
+			(do_not_autoplace no)
+			(effects
+				(font
+					(size 1.27 1.27)
+				)
+			)
+		)
+		(property "Datasheet" ""
+			(at 90.17 72.39 0)
 			(hide yes)
 			(show_name no)
@@
 		)
 		(property "Description" "Power symbol creates a global label with name \"+3.3V\""
-			(at 52.07 67.31 0)
+			(at 90.17 72.39 0)
 			(hide yes)
 			(show_name no)
@@
 	(symbol
 		(lib_id "power:GND")
-		(at 52.07 87.63 0)
+		(at 90.17 92.71 0)
 		(unit 1)
 		(body_style 1)
@@
 		(fields_autoplaced yes)
 		(property "Reference" "#PWR070"
-			(at 52.07 93.98 0)
+			(at 90.17 99.06 0)
 			(hide yes)
 			(show_name no)
@@
 		)
 		(property "Value" "GND"
-			(at 52.07 92.71 0)
+			(at 90.17 97.79 0)
 			(show_name no)
 			(do_not_autoplace no)
@@
 		)
 		(property "Footprint" ""
-			(at 52.07 87.63 0)
-			(hide yes)
-			(show_name no)
-			(do_not_autoplace no)
-			(effects
-				(font
-					(size 1.27 1.27)
-				)
-			)
-		)
-		(property "Datasheet" ""
-			(at 52.07 87.63 0)
+			(at 90.17 92.71 0)
+			(hide yes)
+			(show_name no)
+			(do_not_autoplace no)
+			(effects
+				(font
+					(size 1.27 1.27)
+				)
+			)
+		)
+		(property "Datasheet" ""
+			(at 90.17 92.71 0)
 			(hide yes)
 			(show_name no)
@@
 		)
 		(property "Description" "Power symbol creates a global label with name \"GND\" , ground"
-			(at 52.07 87.63 0)
+			(at 90.17 92.71 0)
 			(hide yes)
 			(show_name no)
@@
 	(symbol
 		(lib_id "Display_Graphic:ER_OLEDM0.91_1x-I2C")
-		(at 52.07 77.47 0)
+		(at 90.17 82.55 0)
 		(unit 1)
 		(body_style 1)
@@
 		(fields_autoplaced yes)
 		(property "Reference" "U7"
-			(at 60.96 78.7401 0)
+			(at 99.06 83.8201 0)
 			(show_name no)
 			(do_not_autoplace no)
@@
 		)
 		(property "Value" "ER_OLEDM0.91_1x-I2C"
-			(at 60.96 76.2001 0)
+			(at 99.06 81.2801 0)
 			(show_name no)
 			(do_not_autoplace no)
@@
 		)
 		(property "Footprint" "Connector_PinHeader_2.54mm:PinHeader_1x04_P2.54mm_Vertical"
-			(at 70.104 90.17 0)
+			(at 108.204 95.25 0)
 			(hide yes)
 			(show_name no)
@@
 		)
 		(property "Datasheet" "https://www.buydisplay.com/download/manual/ER-OLEDM0.91-1_Datasheet.pdf"
-			(at 94.742 92.202 0)
+			(at 132.842 97.282 0)
 			(hide yes)
 			(show_name no)
@@
 		)
 		(property "Description" "SSD1306 OLED module, 0.91 inch, 128x32, I2C"
-			(at 78.74 94.234 0)
-			(hide yes)
-			(show_name no)
+			(at 116.84 99.314 0)
+			(hide yes)
+			(show_name no)

Commit message: Update KiCad project files
Parts:
- added C27, C33: 100nf, Capacitor_SMD:C_0805_2012Metric, symbol Device:C
- renumbered J21 to J8, J22 to J9, R31 to R41, R32 to R42, U7 to U6
Connections:
- net +3V3: now also C27.1, C33.1
- net GND: now also C27.2, C33.2
Other:
- moved on the sheet: U6

Commit message: Remove unused schematic files, lock files, and backup directories
Parts:
- removed J8: Oled SSD1306 128x32, Connector_PinHeader_2.54mm:PinHeader_2x03_P2.54mm_Vertical, symbol Connector_Generic:Conn_01x06
- added J5: Oled SSD1306 128x32, Connector_PinHeader_2.54mm:PinHeader_2x03_P2.54mm_Vertical, symbol Connector_Generic:Conn_02x03_Odd_Even
- U6: footprint Connector_PinHeader_2.54mm:PinHeader_1x04_P2.54mm_Vertical -> kiC:LCD_OLED_128X64_1.3_I2C
Connections:
- net +3.3V: now also J5.1 (Pin_1)
- net +5V: now also J5.2 (Pin_2), J5.4 (Pin_4)
- net GND: now also J5.6 (Pin_6)
- net scl: now also J5.5 (Pin_5)
- net sda: now also J5.3 (Pin_3)

Commit message: Update all schematic files and project
Connections:
- net +3.3V is gone; now on net +3V3: J5.1 (Pin_1), J9.2 (Pin_2), U6.2 (VCC)
Other:
- moved on the sheet: U6

Commit message: Update all schematic files and project
Connections:
- net scl renamed SCL
- net sda renamed SDA
Changed lines of the file:
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@@
 	(wire
 		(pts
-			(xy 110.49 134.62) (xy 110.49 137.16)
+			(xy 40.64 97.79) (xy 48.26 97.79)
+		)
+		(stroke
+			(width 0)
+			(type default)
+		)
+	)
+	(wire
+		(pts
+			(xy 110.49 134.62) (xy 110.49 138.43)
 		)
 		(stroke
@@
 	(wire
 		(pts
+			(xy 96.52 138.43) (xy 110.49 138.43)
+		)
+		(stroke
+			(width 0)
+			(type default)
+		)
+	)
+	(wire
+		(pts
 			(xy 163.83 133.35) (xy 177.8 133.35)
 		)
@@
 	(wire
 		(pts
+			(xy 208.28 93.98) (xy 200.66 93.98)
+		)
+		(stroke
+			(width 0)
+			(type default)
+		)
+	)
+	(wire
+		(pts
+			(xy 200.66 96.52) (xy 222.25 96.52)
+		)
+		(stroke
+			(width 0)
+			(type default)
+		)
+	)
+	(wire
+		(pts
+			(xy 208.28 90.17) (xy 208.28 93.98)
+		)
+		(stroke
+			(width 0)
+			(type default)
+		)
+	)
+	(wire
+		(pts
+			(xy 182.88 128.27) (xy 182.88 133.35)
+		)
+		(stroke
+			(width 0)
+			(type default)
+		)
+	)
+	(wire
+		(pts
+			(xy 212.09 90.17) (xy 208.28 90.17)
+		)
+		(stroke
+			(width 0)
+			(type default)
+		)
+	)
+	(wire
+		(pts
+			(xy 165.1 73.66) (xy 157.48 73.66)
+		)
+		(stroke
+			(width 0)
+			(type default)
+		)
+	)
+	(wire
+		(pts
 			(xy 43.18 92.71) (xy 48.26 92.71)
 		)
@@
 	(wire
 		(pts
-			(xy 208.28 93.98) (xy 200.66 93.98)
-		)
-		(stroke
-			(width 0)
-			(type default)
-		)
-	)
-	(wire
-		(pts
-			(xy 200.66 96.52) (xy 222.25 96.52)
-		)
-		(stroke
-			(width 0)
-			(type default)
-		)
-	)
-	(wire
-		(pts
-			(xy 208.28 90.17) (xy 208.28 93.98)
-		)
-		(stroke
-			(width 0)
-			(type default)
-		)
-	)
-	(wire
-		(pts
-			(xy 182.88 128.27) (xy 182.88 133.35)
-		)
-		(stroke
-			(width 0)
-			(type default)
-		)
-	)
-	(wire
-		(pts
-			(xy 212.09 90.17) (xy 208.28 90.17)
-		)
-		(stroke
-			(width 0)
-			(type default)
-		)
-	)
-	(wire
-		(pts
-			(xy 165.1 73.66) (xy 157.48 73.66)
-		)
-		(stroke
-			(width 0)
-			(type default)
-		)
-	)
-	(wire
-		(pts
-			(xy 110.49 137.16) (xy 96.52 137.16)
-		)
-		(stroke
-			(width 0)
-			(type default)
-		)
-	)
-	(wire
-		(pts
 			(xy 137.16 78.74) (xy 144.78 78.74)
 		)
@@
 		(pts
 			(xy 58.42 107.95) (xy 58.42 105.41)
-		)
-		(stroke
-			(width 0)
-			(type default)
-		)
-	)
-	(wire
-		(pts
-			(xy 41.91 97.79) (xy 48.26 97.79)
 		)
 		(stroke
@@
 	)
 	(label "SCL"
-		(at 45.72 92.71 180)
+		(at 43.18 92.71 180)
 		(effects
 			(font
@@
 	)
 	(label "SDA"
-		(at 105.41 137.16 180)
+		(at 104.14 138.43 180)
 		(effects
 			(font
@@
 	)
 	(label "SDA"
-		(at 44.45 97.79 180)
+		(at 40.64 97.79 180)
 		(effects
 			(font
@@
 		)
 	)
-	(hierarchical_label "sda"
-		(shape input)
-		(at 96.52 137.16 180)
+	(hierarchical_label "SDA"
+		(shape input)
+		(at 96.52 138.43 180)
 		(effects
 			(font
@@
 		)
 	)
-	(hierarchical_label "scl"
+	(hierarchical_label "SCL"
 		(shape input)
 		(at 83.82 124.46 180)

Commit message: Actualización de esquema y PCB del proyecto ESP32C6 Xiaozhi
Parts:
- U6: footprint kiC:LCD_OLED_128X64_1.3_I2C -> kiC:SSD1306_No_Mounting_whitout_Holes
Changed lines of the file:
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@@
 			)
 		)
-		(property "Footprint" "kiC:LCD_OLED_128X64_1.3_I2C"
+		(property "Footprint" "kiC:SSD1306_No_Mounting_whitout_Holes"
 			(at 76.454 107.95 0)
 			(hide yes)
