File: display.kicad_sch (KiCad schematic)
At the start: 7 parts, among them J5 Oled SSD1306 128x32, J9 Adafruit ST7789, U6 ER_OLEDM0.91_1x-I2C

Commit message: Actualizaciones para versión single ESP32C6
Parts:
- U6: footprint kiC:SSD1306_No_Mounting_whitout_Holes -> Connector_PinHeader_2.54mm:PinHeader_1x04_P2.54mm_Vertical
Changed lines of the file:
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@@
 			)
 		)
-		(property "Footprint" "kiC:SSD1306_No_Mounting_whitout_Holes"
+		(property "Footprint" "Connector_PinHeader_2.54mm:PinHeader_1x04_P2.54mm_Vertical"
 			(at 76.454 107.95 0)
 			(hide yes)

Commit message: Update KiCad schematics/PCB and project files
Parts:
- U6: value ER_OLEDM0.91_1x-I2C -> SS1306_OLEDM0.91_1x-I2C
Changed lines of the file:
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@@
 	(wire
 		(pts
-			(xy 58.42 83.82) (xy 55.88 83.82)
+			(xy 96.52 138.43) (xy 110.49 138.43)
 		)
 		(stroke
@@
 	(wire
 		(pts
-			(xy 58.42 107.95) (xy 55.88 107.95)
+			(xy 163.83 133.35) (xy 177.8 133.35)
 		)
 		(stroke
@@
 	(wire
 		(pts
-			(xy 96.52 138.43) (xy 110.49 138.43)
+			(xy 137.16 76.2) (xy 144.78 76.2)
 		)
 		(stroke
@@
 	(wire
 		(pts
-			(xy 163.83 133.35) (xy 177.8 133.35)
+			(xy 208.28 93.98) (xy 200.66 93.98)
 		)
 		(stroke
@@
 	(wire
 		(pts
-			(xy 137.16 76.2) (xy 144.78 76.2)
+			(xy 200.66 96.52) (xy 222.25 96.52)
 		)
 		(stroke
@@
 	(wire
 		(pts
-			(xy 208.28 93.98) (xy 200.66 93.98)
+			(xy 208.28 90.17) (xy 208.28 93.98)
 		)
 		(stroke
@@
 	(wire
 		(pts
-			(xy 200.66 96.52) (xy 222.25 96.52)
+			(xy 182.88 128.27) (xy 182.88 133.35)
 		)
 		(stroke
@@
 	(wire
 		(pts
-			(xy 208.28 90.17) (xy 208.28 93.98)
+			(xy 212.09 90.17) (xy 208.28 90.17)
 		)
 		(stroke
@@
 	(wire
 		(pts
-			(xy 182.88 128.27) (xy 182.88 133.35)
+			(xy 165.1 73.66) (xy 157.48 73.66)
 		)
 		(stroke
@@
 	(wire
 		(pts
-			(xy 212.09 90.17) (xy 208.28 90.17)
+			(xy 43.18 92.71) (xy 48.26 92.71)
 		)
 		(stroke
@@
 	(wire
 		(pts
-			(xy 165.1 73.66) (xy 157.48 73.66)
+			(xy 137.16 78.74) (xy 144.78 78.74)
 		)
 		(stroke
@@
 	(wire
 		(pts
-			(xy 43.18 92.71) (xy 48.26 92.71)
+			(xy 58.42 107.95) (xy 58.42 105.41)
 		)
 		(stroke
@@
 	(wire
 		(pts
-			(xy 137.16 78.74) (xy 144.78 78.74)
+			(xy 83.82 124.46) (xy 96.52 124.46)
 		)
 		(stroke
@@
 	(wire
 		(pts
-			(xy 58.42 107.95) (xy 58.42 105.41)
-		)
-		(stroke
-			(width 0)
-			(type default)
-		)
-	)
-	(wire
-		(pts
-			(xy 83.82 124.46) (xy 96.52 124.46)
-		)
-		(stroke
-			(width 0)
-			(type default)
-		)
-	)
-	(wire
-		(pts
-			(xy 58.42 83.82) (xy 58.42 85.09)
+			(xy 58.42 81.28) (xy 58.42 85.09)
 		)
 		(stroke
@@
 	(symbol
 		(lib_id "power:+3V3")
-		(at 55.88 83.82 0)
+		(at 58.42 81.28 0)
 		(unit 1)
 		(body_style 1)
@@
 		(fields_autoplaced yes)
 		(property "Reference" "#PWR071"
-			(at 55.88 87.63 0)
+			(at 58.42 85.09 0)
 			(hide yes)
 			(show_name no)
@@
 		)
 		(property "Value" "+3V3"
-			(at 55.88 78.74 0)
+			(at 58.42 76.2 0)
 			(show_name no)
 			(do_not_autoplace no)
@@
 		)
 		(property "Footprint" ""
-			(at 55.88 83.82 0)
+			(at 58.42 81.28 0)
 			(hide yes)
 			(show_name no)
@@
 		)
 		(property "Datasheet" ""
-			(at 55.88 83.82 0)
+			(at 58.42 81.28 0)
 			(hide yes)
 			(show_name no)
@@
 		)
 		(property "Description" "Power symbol creates a global label with name \"+3V3\""
-			(at 55.88 83.82 0)
+			(at 58.42 81.28 0)
 			(hide yes)
 			(show_name no)
@@
 	(symbol
 		(lib_id "power:GND")
-		(at 55.88 107.95 0)
+		(at 58.42 107.95 0)
 		(unit 1)
 		(body_style 1)
@@
 		(fields_autoplaced yes)
 		(property "Reference" "#PWR068"
-			(at 55.88 114.3 0)
+			(at 58.42 114.3 0)
 			(hide yes)
 			(show_name no)
@@
 		)
 		(property "Value" "GND"
-			(at 55.88 113.03 0)
+			(at 58.42 113.03 0)
 			(show_name no)
 			(do_not_autoplace no)
@@
 		)
 		(property "Footprint" ""
-			(at 55.88 107.95 0)
+			(at 58.42 107.95 0)
 			(hide yes)
 			(show_name no)
@@
 		)
 		(property "Datasheet" ""
-			(at 55.88 107.95 0)
+			(at 58.42 107.95 0)
 			(hide yes)
 			(show_name no)
@@
 		)
 		(property "Description" "Power symbol creates a global label with name \"GND\" , ground"
-			(at 55.88 107.95 0)
+			(at 58.42 107.95 0)
 			(hide yes)
 			(show_name no)
@@
 		(fields_autoplaced yes)
 		(property "Reference" "U6"
-			(at 67.31 96.5201 0)
+			(at 67.31 93.9799 0)
 			(show_name no)
 			(do_not_autoplace no)
@@
 			)
 		)
-		(property "Value" "ER_OLEDM0.91_1x-I2C"
-			(at 67.31 93.9801 0)
-			(show_name no)
-			(do_not_autoplace no)
+		(property "Value" "SS1306_OLEDM0.91_1x-I2C"
+			(at 67.31 96.5199 0)
+			(show_name no)
+			(do_not_autoplace no)

Commit message: add files update
Parts:
- C33: value 100nf -> 1uf
- J5: now left out of the parts list
Changed lines of the file:
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@@
 		(body_style 1)
 		(exclude_from_sim no)
-		(in_bom yes)
-		(on_board yes)
-		(in_pos_files yes)
+		(in_bom no)
+		(on_board yes)
+		(in_pos_files no)
 		(dnp no)
 		(property "Reference" "J5"
@@
 			)
 		)
-		(property "Description" ""
-			(at 195.58 101.6 0)
+		(property "Description" "Display LCD ST7789 240x240 pixels"
+			(at 208.534 112.776 0)
 			(show_name no)
 			(do_not_autoplace no)
@@
 		(fields_autoplaced yes)
 		(property "Reference" "C33"
-			(at 181.61 135.89 0)
+			(at 181.61 135.8899 0)
 			(show_name no)
 			(do_not_autoplace no)
@@
 			)
 		)
-		(property "Value" "100nf"
-			(at 181.61 138.43 0)
+		(property "Value" "1uf"
+			(at 181.61 138.4299 0)
 			(show_name no)
 			(do_not_autoplace no)
@@
 			)
 		)
-		(property "Description" "SSD1306 OLED module, 0.91 inch, 128x32, I2C"
+		(property "Description" "SSD1306 OLED module, 0.91 inch, 128x64, I2C"
 			(at 85.09 112.014 0)
 			(hide yes)

Commit message: Actualización de esquemas y PCB con datos LCSC y librerías JLC
- Añade propiedades LCSC a los símbolos de las hojas de esquema
- Actualiza las hojas TXS0108E, display, esp32_c6, ft232, inmp441,
  led_sw_gpio, max98357a, micro_sd, power_supply y el esquema raíz
- Reorganiza el PCB (footprints, jumpers y nets) y actualiza el proyecto
- Incluye las librerías locales JLCImport (símbolos, huellas y modelos 3D)
  y las entradas correspondientes en fp-lib-table y sym-lib-table
- Añade la documentación técnica en docs/ y el archivo de posiciones
  esp32_xiaozhi-all.pos
- Elimina los ZIP generados gebers.zip y production.zip
Parts:
- C27: LCSC (none) -> C1525
- C33: LCSC (none) -> C28323
- J5: LCSC (none) -> C9900045120
- J9: LCSC (none) -> C9900247203; now left out of the parts list
- R41, R42: LCSC (none) -> C4190
- U6: now left out of the parts list
Changed lines of the file:
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@@
+			)
+		)
+		(property "LCSC" "C1525"
+			(at 163.83 137.16 0)
+			(hide yes)
+			(show_name no)
+			(do_not_autoplace no)
+			(effects
+				(font
+					(size 1.27 1.27)
+				)
 			)
 		)
@@
 			)
 		)
+		(property "LCSC" "C9900045120"
+			(at 149.86 76.2 0)
+			(hide yes)
+			(show_name no)
+			(do_not_autoplace no)
+			(effects
+				(font
+					(size 1.27 1.27)
+				)
+			)
+		)
 		(pin "3"
 		)
@@
 		(body_style 1)
 		(exclude_from_sim no)
-		(in_bom yes)
-		(on_board yes)
-		(in_pos_files yes)
+		(in_bom no)
+		(on_board yes)
+		(in_pos_files no)
 		(dnp no)
 		(property "Reference" "J9"
@@
 		(property "Description" "Display LCD ST7789 240x240 pixels"
 			(at 208.534 112.776 0)
+			(show_name no)
+			(do_not_autoplace no)
+			(effects
+				(font
+					(size 1.27 1.27)
+				)
+			)
+		)
+		(property "LCSC" "C9900247203"
+			(at 195.58 101.6 0)
+			(hide yes)
 			(show_name no)
 			(do_not_autoplace no)
@@
 			)
 		)
+		(property "LCSC" "C28323  "
+			(at 177.8 137.16 0)
+			(hide yes)
+			(show_name no)
+			(do_not_autoplace no)
+			(effects
+				(font
+					(size 1.27 1.27)
+				)
+			)
+		)
 		(pin "1"
 		)
@@
 			)
 		)
+		(property "LCSC" "C4190"
+			(at 110.49 130.81 0)
+			(hide yes)
+			(show_name no)
+			(do_not_autoplace no)
+			(effects
+				(font
+					(size 1.27 1.27)
+				)
+			)
+		)
 		(pin "1"
 		)
@@
 			)
 		)
+		(property "LCSC" "C4190"
+			(at 96.52 120.65 0)
+			(hide yes)
+			(show_name no)
+			(do_not_autoplace no)
+			(effects
+				(font
+					(size 1.27 1.27)
+				)
+			)
+		)
 		(pin "1"
 		)
@@
 		(body_style 1)
 		(exclude_from_sim no)
-		(in_bom yes)
-		(on_board yes)
-		(in_pos_files yes)
+		(in_bom no)
+		(on_board yes)
+		(in_pos_files no)
 		(dnp no)
 		(fields_autoplaced yes)

Commit message: Actualización de esquemas, PCB y librerías
Parts:
- added C58, C61, C62, C63, C64: 100nf, Capacitor_SMD:C_0402_1005Metric, symbol Device:C
- added C59, C60: 4.7uf, Capacitor_SMD:C_0805_2012Metric, symbol Device:C
- added J14: Adafruit ST7789, Connector_PinHeader_2.54mm:PinHeader_1x08_P2.54mm_Vertical, symbol Connector:Conn_01x07_Pin
- added JP13, JP15, JP16: NL, Jumper:SolderJumper-2_P1.3mm_Open_RoundedPad1.0x1.5mm, symbol Jumper:Jumper_2_Open
- added L8: 100mh, Inductor_SMD:L_1206_3216Metric, symbol Device:L
- added Q7: Q_NPN_BCE, Package_TO_SOT_SMD:SOT-23W, symbol Device:Q_NPN_BCE
- added R30: 2k2, Resistor_SMD:R_0805_2012Metric, symbol Device:R
- added R49: 10k, Resistor_SMD:R_0805_2012Metric, symbol Device:R
- added U14: LM1117DT-3.3, kiC:TO-252-3_TabPin2, symbol Regulator_Linear:LM1117DT-3.3
- added U3: HS20HS072RX, JLCImport:OLED-SMD_HS20HS072RX, symbol HS20HS072RX:HS20HS072RX
- C27: LCSC C1525 -> C28233
- R41, R42: LCSC C4190 -> C17520
- U6: LCSC (none) -> C5248080; now in the parts list
Connections:
- net GND: now also C58.1, C59.1, C60.1, C61.1, C62.1, C63.1, C64.1, J14.1 (Pin_1), JP16.2 (B), Q7.3 (E), U14.1 (GND1), U3.1 (GND), U3.12 (GND)
- new net: JP15.2 (B), JP16.1 (A), U3.3 (RS)
- new net: J14.3 (Pin_3), U3.5 (SDA)
- new net: J14.4 (Pin_4), U3.4 (SCL)
- new net: J14.5 (Pin_5), U3.6 (RST)
- new net: J14.6 (Pin_6), U3.2 (CS)
- new net: J14.7 (Pin_7), R30.1
- new net: Q7.2 (C), R49.2, U3.11 (K)
- new net: JP13.2 (B), U3.8 (I/O-VCC)
- new net: C60.2, C64.2, L8.1, U14.2 (VO)
- new net: Q7.1 (B), R30.2
- new net +VCC_3.3: C58.2, C61.2, C62.2, JP13.1 (A), JP15.1 (A), L8.2, R49.1, U3.10 (A), U3.9 (VCC)
- new net +VCC_5: C59.2, C63.2, J14.2 (Pin_2), U14.3 (VI)
- no-connect marks 0 -> 1
Other:
- moved on the sheet: C27, C33, J5, J9, R41, R42, U6

Commit message: update epaper and mt48
Connections:
- net _RS: now reaches JP15.2 (B), JP16.1 (A), U3.3 (RS)
- net _SDA: now reaches J14.3 (Pin_3), U3.5 (SDA)
- net _SCL: now reaches J14.4 (Pin_4), U3.4 (SCL)
- net _RST: now reaches J14.5 (Pin_5), U3.6 (RST)
- net _CS: now reaches J14.6 (Pin_6), U3.2 (CS)
Other:
- added sheet epaper (epaper.kicad_sch)
Changed lines of the file:
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@@
 		)
 	)
+	(label "_SCL"
+		(at 59.69 48.26 0)
+		(effects
+			(font
+				(size 1.27 1.27)
+			)
+			(justify left bottom)
+		)
+	)
 	(label "+VCC_5"
 		(at 40.64 43.18 0)
@@
 		)
 	)
+	(label "_RST"
+		(at 59.69 50.8 0)
+		(effects
+			(font
+				(size 1.27 1.27)
+			)
+			(justify left bottom)
+		)
+	)
 	(label "SCL"
 		(at 35.56 121.92 180)
@@
 		)
 	)
+	(label "_CS"
+		(at 62.23 53.34 0)
+		(effects
+			(font
+				(size 1.27 1.27)
+			)
+			(justify left bottom)
+		)
+	)
 	(label "+VCC_3.3"
 		(at 205.74 30.48 0)
@@
 		)
 	)
+	(label "_SDA"
+		(at 59.69 45.72 0)
+		(effects
+			(font
+				(size 1.27 1.27)
+			)
+			(justify left bottom)
+		)
+	)
 	(label "+VCC_5"
 		(at 160.02 25.4 0)
@@
 		)
 	)
+	(label "_RS"
+		(at 87.63 46.99 0)
+		(effects
+			(font
+				(size 1.27 1.27)
+			)
+			(justify left bottom)
+		)
+	)
 	(label "SCL"
 		(at 125.73 157.48 180)
@@
 				)
 			)
+		)
+	)
+	(sheet
+		(at 153.035 71.755)
+		(size 62.865 48.26)
+		(exclude_from_sim no)
+		(in_bom yes)
+		(on_board yes)
+		(dnp no)
+		(fields_autoplaced yes)
+		(stroke
+			(width 0.1524)
+			(type solid)
+		)
+		(fill
+			(color 0 0 0 0)
+		)
+		(property "Sheetname" "epaper"
+			(at 153.035 71.0434 0)
+			(show_name no)
+			(do_not_autoplace no)
+			(effects
+				(font
+					(size 1.27 1.27)
+				)
+				(justify left bottom)
+			)
+		)
+		(property "Sheetfile" "epaper.kicad_sch"
+			(at 153.035 120.5996 0)
+			(show_name no)
+			(do_not_autoplace no)
+			(effects
+				(font
+					(size 1.27 1.27)
+				)
+				(justify left top)
+			)
+		)
+		(instances
+			(project "esp32_xiaozhi"
+				(path "/cae338e8-f342-43cb-b99a-a0486629133c/c0550844-e74d-4e5d-964f-3b0622860ba1"
+					(page "10")
+				)
+			)

Commit message: actualizacion  de pcb logic , rpi
Parts:
- U6: now left out of the parts list
Changed lines of the file:
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@@
 		(body_style 1)
 		(exclude_from_sim no)
-		(in_bom yes)
+		(in_bom no)
 		(on_board yes)
-		(in_pos_files yes)
+		(in_pos_files no)
 		(dnp no)
 		(fields_autoplaced yes)

Commit message: correccion de numero de partes de componentes
Parts:
- JP13, JP15, JP16: now left out of the parts list
- L8: value 100mh -> 60Ω@100MHz
Changed lines of the file:
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@@
 		(body_style 1)
 		(exclude_from_sim no)
-		(in_bom yes)
-		(on_board yes)
-		(in_pos_files yes)
+		(in_bom no)
+		(on_board yes)
+		(in_pos_files no)
 		(dnp no)
 		(property "Reference" "JP16"
@@
 			)
 		)
-		(property "Value" "100mh"
+		(property "Value" "60Ω@100MHz"
 			(at 204.47 33.02 90)
 			(hide yes)
@@
 			)
 		)
-		(property "Description" "1 60Ω@100MHz ±25% 1206 Ferrite Beads ROHS"
+		(property "Description" "60Ω@100MHz ±25% 1206 Ferrite Beads ROHS"
 			(at 202.946 16.51 90)
 			(hide yes)
@@
 		(body_style 1)
 		(exclude_from_sim no)
-		(in_bom yes)
-		(on_board yes)
-		(in_pos_files yes)
+		(in_bom no)
+		(on_board yes)
+		(in_pos_files no)
 		(dnp no)
 		(property "Reference" "JP13"
@@
 		(body_style 1)
 		(exclude_from_sim no)
-		(in_bom yes)
-		(on_board yes)
-		(in_pos_files yes)
+		(in_bom no)
+		(on_board yes)
+		(in_pos_files no)
 		(dnp no)
 		(property "Reference" "JP15"
