File: display.kicad_sch (KiCad schematic)
At the start: 24 parts, among them J14 Adafruit ST7789, J5 Oled SSD1306 128x32, J9 Adafruit ST7789, Q7 Q_NPN_BCE, U14 LM1117DT-3.3, U3 HS20HS072RX, U6 SS1306_OLEDM0.91_1x-I2C

Commit message: add update
Parts:
- U3: LCSC (none) -> C5329582
Changed lines of the file:
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@@
+			)
+		)
+		(property "LCSC" "C5329582"
+			(at 101.6 55.88 0)
+			(hide yes)
+			(show_name no)
+			(do_not_autoplace no)
+			(effects
+				(font
+					(size 1.27 1.27)
+				)
 			)
 		)

Commit message: correccion de partes
Parts:
- U14: value LM1117DT-3.3 -> LM1117MDT-3.3/TR; LCSC C969102 -> C498159
- U3: footprint JLCImport:OLED-SMD_HS20HS072RX -> Libraries:OLED-SMD_HS20HS072RX
Changed lines of the file:
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@@
 			)
 		)
-		(property "Footprint" "JLCImport:OLED-SMD_HS20HS072RX"
+		(property "Footprint" "Libraries:OLED-SMD_HS20HS072RX"
 			(at 101.6 77.47 0)
 			(hide yes)
@@
 			)
 		)
-		(property "Value" "LM1117DT-3.3"
+		(property "Value" "LM1117MDT-3.3/TR"
 			(at 176.53 26.67 0)
 			(show_name no)
@@
 			)
 		)
-		(property "LCSC" "C969102"
+		(property "LCSC" "C498159"
 			(at 176.53 30.48 0)
 			(hide yes)
