File: board.kicad_sch (KiCad schematic)
At the start: 8 parts, among them U10 LM393, U11 PIN_HEADER_36, U13 TL431DBZ

Commit message: Actualizaciones para versión single ESP32C6
Parts:
- added R74, R75: 2k2, Resistor_SMD:R_0805_2012Metric, symbol Device:R
Connections:
- net PIN_25 is gone; now on net IN1-: U11.25 (P25)
- net PIN_26 is gone; now on net IN2-: U11.26 (P26)
- net PIN_27 is gone; now on net IN2+: U11.27 (P27)
- net PIN_28 is gone; now on net PIN_18: U11.28 (P28)
- net PIN_29 is gone; now on net OUT2: U11.29 (P29)
- net PIN_30 is gone; now on net OUT1: U11.30 (P30)
- net GND: now also R74.1, R75.1
- net IN2+: now also R74.2
- net OUT1: no longer U11.20 (P20)
- net OUT2: no longer U11.19 (P19)
- net IN1+ renamed PIN_18
- net PIN_18: now also R75.2
- net PIN_21: no longer names the net of U11.21 (P21)
- net PIN_22: no longer names the net of U11.22 (P22)
- net PIN_23: no longer names the net of U11.23 (P23)
- net PIN_24: no longer names the net of U11.24 (P24)
- net PIN_7: no longer names the net of U11.7 (P7)
- net PIN_8: no longer names the net of U11.8 (P8)
- net PIN_9: no longer names the net of U11.9 (P9)
Other:
- moved on the sheet: R72, R73, U10C
