File: led_sw_gpio.kicad_sch (KiCad schematic)
At the start: 31 parts, among them Q6 2N7002, SW3 up, SW4 down, SW5 left, SW6 rigth, SW7 up, SW8 down

Commit message: Update all schematic files and project
Parts:
- added D13: LED, Diode_SMD:D_0805_2012Metric, symbol Device:LED
- added R39: 2k2, Resistor_SMD:R_0805_2012Metric, symbol Device:R
Connections:
- net +3V3: now also D13.2 (A)
- net GND: now also R39.1
- net led3: now also D3.2 (A); no longer D3.1 (K)
- net led4: now also D4.2 (A); no longer D4.1 (K)
- net led5: now also D5.2 (A); no longer D5.1 (K)
- net led6: now also D6.2 (A); no longer D6.1 (K)
- net at R28.2: now also D4.1 (K); no longer D4.2 (A)
- net at R29.2: now also D5.1 (K); no longer D5.2 (A)
- net at R30.2: now also D6.1 (K); no longer D6.2 (A)
- net at R27.2: now also D3.1 (K); no longer D3.2 (A)
- new net: D13.1 (K), R39.2
Other:
- moved on the sheet: D3, D4, D5, D6, R33, R34

Commit message: Update schematics, PCB, and project files
Other:
- moved on the sheet: D7, R40
Changed lines of the file:
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@@
 	)
 	(no_connect
-		(at 374.65 220.98)
+		(at 375.92 220.98)
 	)
 	(wire
@@
 	(wire
 		(pts
-			(xy 356.87 218.44) (xy 359.41 218.44)
+			(xy 356.87 220.98) (xy 360.68 220.98)
 		)
 		(stroke
@@
 	(wire
 		(pts
-			(xy 367.03 228.6) (xy 367.03 233.68)
+			(xy 368.3 228.6) (xy 368.3 233.68)
 		)
 		(stroke
@@
 	(wire
 		(pts
-			(xy 367.03 233.68) (xy 365.76 233.68)
+			(xy 368.3 233.68) (xy 365.76 233.68)
 		)
 		(stroke
@@
 	(wire
 		(pts
-			(xy 367.03 210.82) (xy 367.03 213.36)
+			(xy 368.3 210.82) (xy 368.3 213.36)
 		)
 		(stroke
@@
 	(wire
 		(pts
-			(xy 307.34 201.93) (xy 307.34 200.66)
-		)
-		(stroke
-			(width 0)
-			(type default)
-		)
-	)
-	(wire
-		(pts
-			(xy 359.41 218.44) (xy 359.41 220.98)
+			(xy 307.34 201.93) (xy 307.34 198.12)
 		)
 		(stroke
@@
 	(wire
 		(pts
-			(xy 367.03 210.82) (xy 369.57 210.82)
+			(xy 125.73 105.41) (xy 125.73 116.84)
 		)
 		(stroke
@@
 	(wire
 		(pts
-			(xy 125.73 105.41) (xy 125.73 116.84)
+			(xy 234.95 101.6) (xy 234.95 114.3)
 		)
 		(stroke
@@
 	(wire
 		(pts
-			(xy 234.95 101.6) (xy 234.95 114.3)
+			(xy 273.05 154.94) (xy 273.05 143.51)
 		)
 		(stroke
@@
 	(wire
 		(pts
-			(xy 273.05 154.94) (xy 273.05 143.51)
+			(xy 307.34 189.23) (xy 307.34 190.5)
 		)
 		(stroke
@@
 	(global_label "LED_Data_5V"
 		(shape input)
-		(at 307.34 201.93 0)
+		(at 307.34 199.39 0)
 		(fields_autoplaced yes)
 		(effects
@@
 		)
 		(property "Intersheetrefs" "${INTERSHEET_REFS}"
-			(at 322.2993 201.93 0)
+			(at 322.2993 199.39 0)
 			(hide yes)
 			(show_name no)
@@
 	(global_label "LED_Data_5V"
 		(shape input)
-		(at 356.87 218.44 180)
+		(at 356.87 220.98 180)
 		(fields_autoplaced yes)
 		(effects
@@
 		)
 		(property "Intersheetrefs" "${INTERSHEET_REFS}"
-			(at 341.9901 218.44 0)
+			(at 341.9901 220.98 0)
 			(hide yes)
 			(show_name no)
@@
 	(symbol
 		(lib_id "power:+5V")
-		(at 369.57 210.82 0)
+		(at 368.3 210.82 0)
 		(unit 1)
 		(body_style 1)
@@
 		(fields_autoplaced yes)
 		(property "Reference" "#PWR065"
-			(at 369.57 214.63 0)
+			(at 368.3 214.63 0)
 			(hide yes)
 			(show_name no)
@@
 		)
 		(property "Value" "+5V"
-			(at 372.11 209.5499 0)
+			(at 370.84 209.5499 0)
 			(show_name no)
 			(do_not_autoplace no)
@@
 		)
 		(property "Footprint" ""
-			(at 369.57 210.82 0)
+			(at 368.3 210.82 0)
 			(hide yes)
 			(show_name no)
@@
 		)
 		(property "Datasheet" ""
-			(at 369.57 210.82 0)
+			(at 368.3 210.82 0)
 			(hide yes)
 			(show_name no)
@@
 		)
 		(property "Description" ""
-			(at 369.57 210.82 0)
+			(at 368.3 210.82 0)
 			(show_name no)
 			(do_not_autoplace no)
@@
 	(symbol
 		(lib_id "LED:WS2812B")
-		(at 367.03 220.98 0)
+		(at 368.3 220.98 0)
 		(unit 1)
 		(body_style 1)
@@
 		(dnp no)
 		(property "Reference" "D7"
-			(at 362.585 214.63 0)
+			(at 363.855 214.63 0)
 			(show_name no)
 			(do_not_autoplace no)
@@
 		)
 		(property "Value" "WS2812B"
-			(at 372.11 214.63 0)
+			(at 373.38 214.63 0)
 			(show_name no)
 			(do_not_autoplace no)
@@
 		)
 		(property "Footprint" "LED_SMD:LED_WS2812B_PLCC4_5.0x5.0mm_P3.2mm"
-			(at 368.3 228.6 0)
+			(at 369.57 228.6 0)
 			(hide yes)
 			(show_name no)
@@
 		)
 		(property "Datasheet" "https://cdn-shop.adafruit.com/datasheets/WS2812B.pdf"
-			(at 369.57 230.505 0)
+			(at 370.84 230.505 0)
 			(hide yes)
 			(show_name no)
@@
 		)
 		(property "Description" ""
-			(at 367.03 220.98 0)
+			(at 368.3 220.98 0)
 			(show_name no)
 			(do_not_autoplace no)
@@
 		)
 		(property "LCSC Part #" "C2761795"
-			(at 367.03 220.98 0)
+			(at 368.3 220.98 0)
 			(hide yes)
 			(show_name no)
@@
 	(symbol
 		(lib_id "power:+5V")
-		(at 307.34 193.04 0)
+		(at 307.34 189.23 0)
 		(unit 1)
 		(body_style 1)
@@
 		(fields_autoplaced yes)
 		(property "Reference" "#PWR063"
-			(at 307.34 196.85 0)
+			(at 307.34 193.04 0)
 			(hide yes)
 			(show_name no)
@@
 		)
 		(property "Value" "+5V"
-			(at 309.88 191.7699 0)
+			(at 309.88 187.9599 0)
 			(show_name no)
 			(do_not_autoplace no)
@@
 		)
 		(property "Footprint" ""
-			(at 307.34 193.04 0)
+			(at 307.34 189.23 0)
 			(hide yes)
 			(show_name no)
@@
 		)
 		(property "Datasheet" ""
-			(at 307.34 193.04 0)
+			(at 307.34 189.23 0)
 			(hide yes)
 			(show_name no)
@@
 		)
 		(property "Description" ""
-			(at 307.34 193.04 0)
+			(at 307.34 189.23 0)
 			(show_name no)
 			(do_not_autoplace no)
@@
 	(symbol
 		(lib_id "Device:R")
-		(at 307.34 196.85 180)
+		(at 307.34 194.31 180)
 		(unit 1)
 		(body_style 1)
@@
 		(fields_autoplaced yes)
 		(property "Reference" "R40"
-			(at 304.8 198.1201 0)
+			(at 304.8 195.5801 0)
 			(show_name no)
 			(do_not_autoplace no)
@@
 		)
 		(property "Value" "2k2"
-			(at 304.8 195.5801 0)
+			(at 304.8 193.0401 0)
 			(show_name no)
 			(do_not_autoplace no)
@@
 		)
 		(property "Footprint" "Resistor_SMD:R_0805_2012Metric"
-			(at 309.118 196.85 90)
+			(at 309.118 194.31 90)
 			(hide yes)
 			(show_name no)
@@
 		)
 		(property "Datasheet" ""
-			(at 307.34 196.85 0)
+			(at 307.34 194.31 0)
 			(hide yes)
 			(show_name no)
@@
 		)
 		(property "Description" ""
-			(at 307.34 196.85 0)
+			(at 307.34 194.31 0)
 			(show_name no)
 			(do_not_autoplace no)

Commit message: Add PWR_FLAG symbols to all schematic sheets to fix power_pin_not_driven ERC errors
Changed lines of the file:
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@@
+		)
+	)
+	(symbol
+		(lib_id "power:PWR_FLAG")
+		(at 50.0 50.0 0)
+		(unit 1)
+		(body_style 1)
+		(exclude_from_sim no)
+		(in_bom no)
+		(on_board yes)
+		(in_pos_files no)
+		(dnp no)
+		(property "Reference" "#FLG030"
+			(at 50.0 45.0 0)
+			(hide yes)
+			(show_name no)
+			(do_not_autoplace no)
+			(effects
+				(font
+					(size 1.27 1.27)
+				)
+			)
+		)
+		(property "Value" "PWR_FLAG"
+			(at 50.0 55.0 0)
+			(hide yes)
+			(show_name no)
+			(do_not_autoplace no)
+			(effects
+				(font
+					(size 1.27 1.27)
+				)
+			)
+		)
+		(pin "1"
+			(uuid "d2e3f4a5-6789-01bc-def0-123456789015-pin1")
+		)
+		(instances
+			(project "esp32_xiaozhi"
+				(path "/cae338e8-f342-43cb-b99a-a0486629133c/7256592f-47bf-4ef9-8c00-e0996fdaf86a"
+					(reference "#FLG030")
+					(unit 1)
+				)
+			)
+		)
+	)
+	(symbol
+		(lib_id "power:PWR_FLAG")
+		(at 50.0 100.0 0)
+		(unit 1)
+		(body_style 1)
+		(exclude_from_sim no)
+		(in_bom no)
+		(on_board yes)
+		(in_pos_files no)
+		(dnp no)
+		(property "Reference" "#FLG031"
+			(at 50.0 95.0 0)
+			(hide yes)
+			(show_name no)
+			(do_not_autoplace no)
+			(effects
+				(font
+					(size 1.27 1.27)
+				)
+			)
+		)
+		(property "Value" "PWR_FLAG"
+			(at 50.0 105.0 0)
+			(hide yes)
+			(show_name no)
+			(do_not_autoplace no)
+			(effects
+				(font
+					(size 1.27 1.27)
+				)
+			)
+		)
+		(pin "1"
+			(uuid "d2e3f4a5-6789-01bc-def0-123456789016-pin1")
+		)
+		(instances
+			(project "esp32_xiaozhi"
+				(path "/cae338e8-f342-43cb-b99a-a0486629133c/7256592f-47bf-4ef9-8c00-e0996fdaf86a"
+					(reference "#FLG031")
+					(unit 1)
+				)
+			)
+		)
+	)
+	(symbol
+		(lib_id "power:PWR_FLAG")
+		(at 50.0 150.0 0)
+		(unit 1)
+		(body_style 1)
+		(exclude_from_sim no)
+		(in_bom no)
+		(on_board yes)
+		(in_pos_files no)
+		(dnp no)
+		(property "Reference" "#FLG032"
+			(at 50.0 145.0 0)
+			(hide yes)
+			(show_name no)
+			(do_not_autoplace no)
+			(effects
+				(font
+					(size 1.27 1.27)
+				)
+			)
+		)
+		(property "Value" "PWR_FLAG"
+			(at 50.0 155.0 0)
+			(hide yes)
+			(show_name no)
+			(do_not_autoplace no)
+			(effects
+				(font
+					(size 1.27 1.27)
+				)
+			)
+		)
+		(pin "1"
+			(uuid "d2e3f4a5-6789-01bc-def0-123456789017-pin1")
+		)
+		(instances
+			(project "esp32_xiaozhi"
+				(path "/cae338e8-f342-43cb-b99a-a0486629133c/7256592f-47bf-4ef9-8c00-e0996fdaf86a"
+					(reference "#FLG032")
+					(unit 1)
+				)
+			)
 		)
 	)

Commit message: Revert PWR_FLAG additions - remove '??' squares from schematics
Changed lines of the file:
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@@
-		)
-	)
-	(symbol
-		(lib_id "power:PWR_FLAG")
-		(at 50.0 50.0 0)
-		(unit 1)
-		(body_style 1)
-		(exclude_from_sim no)
-		(in_bom no)
-		(on_board yes)
-		(in_pos_files no)
-		(dnp no)
-		(property "Reference" "#FLG030"
-			(at 50.0 45.0 0)
-			(hide yes)
-			(show_name no)
-			(do_not_autoplace no)
-			(effects
-				(font
-					(size 1.27 1.27)
-				)
-			)
-		)
-		(property "Value" "PWR_FLAG"
-			(at 50.0 55.0 0)
-			(hide yes)
-			(show_name no)
-			(do_not_autoplace no)
-			(effects
-				(font
-					(size 1.27 1.27)
-				)
-			)
-		)
-		(pin "1"
-			(uuid "d2e3f4a5-6789-01bc-def0-123456789015-pin1")
-		)
-		(instances
-			(project "esp32_xiaozhi"
-				(path "/cae338e8-f342-43cb-b99a-a0486629133c/7256592f-47bf-4ef9-8c00-e0996fdaf86a"
-					(reference "#FLG030")
-					(unit 1)
-				)
-			)
-		)
-	)
-	(symbol
-		(lib_id "power:PWR_FLAG")
-		(at 50.0 100.0 0)
-		(unit 1)
-		(body_style 1)
-		(exclude_from_sim no)
-		(in_bom no)
-		(on_board yes)
-		(in_pos_files no)
-		(dnp no)
-		(property "Reference" "#FLG031"
-			(at 50.0 95.0 0)
-			(hide yes)
-			(show_name no)
-			(do_not_autoplace no)
-			(effects
-				(font
-					(size 1.27 1.27)
-				)
-			)
-		)
-		(property "Value" "PWR_FLAG"
-			(at 50.0 105.0 0)
-			(hide yes)
-			(show_name no)
-			(do_not_autoplace no)
-			(effects
-				(font
-					(size 1.27 1.27)
-				)
-			)
-		)
-		(pin "1"
-			(uuid "d2e3f4a5-6789-01bc-def0-123456789016-pin1")
-		)
-		(instances
-			(project "esp32_xiaozhi"
-				(path "/cae338e8-f342-43cb-b99a-a0486629133c/7256592f-47bf-4ef9-8c00-e0996fdaf86a"
-					(reference "#FLG031")
-					(unit 1)
-				)
-			)
-		)
-	)
-	(symbol
-		(lib_id "power:PWR_FLAG")
-		(at 50.0 150.0 0)
-		(unit 1)
-		(body_style 1)
-		(exclude_from_sim no)
-		(in_bom no)
-		(on_board yes)
-		(in_pos_files no)
-		(dnp no)
-		(property "Reference" "#FLG032"
-			(at 50.0 145.0 0)
-			(hide yes)
-			(show_name no)
-			(do_not_autoplace no)
-			(effects
-				(font
-					(size 1.27 1.27)
-				)
-			)
-		)
-		(property "Value" "PWR_FLAG"
-			(at 50.0 155.0 0)
-			(hide yes)
-			(show_name no)
-			(do_not_autoplace no)
-			(effects
-				(font
-					(size 1.27 1.27)
-				)
-			)
-		)
-		(pin "1"
-			(uuid "d2e3f4a5-6789-01bc-def0-123456789017-pin1")
-		)
-		(instances
-			(project "esp32_xiaozhi"
-				(path "/cae338e8-f342-43cb-b99a-a0486629133c/7256592f-47bf-4ef9-8c00-e0996fdaf86a"
-					(reference "#FLG032")
-					(unit 1)
-				)
-			)
 		)
 	)

Commit message: Actualización de esquema y PCB del proyecto ESP32C6 Xiaozhi
Parts:
- removed D5: LED, Diode_SMD:D_0805_2012Metric, symbol Device:LED
- removed R29: 2k2, Resistor_SMD:R_0805_2012Metric, symbol Device:R
Connections:
- net led3 is gone; now on net +5V: D3.2 (A)
Changed lines of the file:
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@@
 		(color 0 0 0 0)
 	)
-	(junction
-		(at 102.87 215.9)
-		(diameter 0)
-		(color 0 0 0 0)
-	)
 	(no_connect
 		(at 375.92 220.98)
@@
 	(wire
 		(pts
-			(xy 113.03 215.9) (xy 102.87 215.9)
-		)
-		(stroke
-			(width 0)
-			(type default)
-		)
-	)
-	(wire
-		(pts
 			(xy 302.26 201.93) (xy 307.34 201.93)
 		)
@@
 	(wire
 		(pts
-			(xy 102.87 210.82) (xy 102.87 215.9)
-		)
-		(stroke
-			(width 0)
-			(type default)
-		)
-	)
-	(wire
-		(pts
 			(xy 266.7 130.81) (xy 273.05 130.81)
 		)
@@
 	(wire
 		(pts
-			(xy 102.87 195.58) (xy 102.87 185.42)
-		)
-		(stroke
-			(width 0)
-			(type default)
-		)
-	)
-	(wire
-		(pts
 			(xy 158.75 147.32) (xy 165.1 147.32)
 		)
@@
 	(wire
 		(pts
-			(xy 92.71 215.9) (xy 102.87 215.9)
+			(xy 92.71 215.9) (xy 113.03 215.9)
 		)
 		(stroke
@@
 		)
 	)
-	(hierarchical_label "led5"
-		(shape input)
-		(at 102.87 185.42 0)
-		(effects
-			(font
-				(size 1.27 1.27)
-			)
-			(justify left)
-		)
-	)
-	(hierarchical_label "led3"
-		(shape input)
-		(at 82.55 185.42 0)
-		(effects
-			(font
-				(size 1.27 1.27)
-			)
-			(justify left)
-		)
-	)
 	(symbol
 		(lib_id "Device:R")
@@
 	(symbol
 		(lib_id "Device:LED")
-		(at 102.87 199.39 90)
-		(unit 1)
-		(body_style 1)
-		(exclude_from_sim no)
-		(in_bom yes)
-		(on_board yes)
-		(in_pos_files yes)
-		(dnp no)
-		(fields_autoplaced yes)
-		(property "Reference" "D5"
-			(at 106.68 199.7074 90)
-			(show_name no)
-			(do_not_autoplace no)
-			(effects
-				(font
-					(size 1.27 1.27)
-				)
-				(justify right)
-			)
-		)
-		(property "Value" "LED"
-			(at 106.68 202.2474 90)
-			(show_name no)
-			(do_not_autoplace no)
-			(effects
-				(font
-					(size 1.27 1.27)
-				)
-				(justify right)
-			)
-		)
-		(property "Footprint" "Diode_SMD:D_0805_2012Metric"
-			(at 102.87 199.39 0)
-			(hide yes)
-			(show_name no)
-			(do_not_autoplace no)
-			(effects
-				(font
-					(size 1.27 1.27)
-				)
-			)
-		)
-		(property "Datasheet" ""
-			(at 102.87 199.39 0)
-			(hide yes)
-			(show_name no)
-			(do_not_autoplace no)
-			(effects
-				(font
-					(size 1.27 1.27)
-				)
-			)
-		)
-		(property "Description" "Light emitting diode"
-			(at 102.87 199.39 0)
-			(hide yes)
-			(show_name no)
-			(do_not_autoplace no)
-			(effects
-				(font
-					(size 1.27 1.27)
-				)
-			)
-		)
-		(property "Sim.Pins" "1=K 2=A"
-			(at 102.87 199.39 0)
-			(hide yes)
-			(show_name no)
-			(do_not_autoplace no)
-			(effects
-				(font
-					(size 1.27 1.27)
-				)
-			)
-		)
-		(pin "1"
-		)
-		(pin "2"
-		)
-		(instances
-			(project "esp32_xiaozhi"
-				(path "/cae338e8-f342-43cb-b99a-a0486629133c/7256592f-47bf-4ef9-8c00-e0996fdaf86a"
-					(reference "D5")
-					(unit 1)
-				)
-			)
-		)
-	)
-	(symbol
-		(lib_id "Device:LED")
 		(at 92.71 199.39 90)
 		(unit 1)
@@
 	(symbol
 		(lib_id "Device:R")
-		(at 102.87 207.01 180)
-		(unit 1)
-		(body_style 1)
-		(exclude_from_sim no)
-		(in_bom yes)
-		(on_board yes)
-		(in_pos_files yes)
-		(dnp no)
-		(fields_autoplaced yes)
-		(property "Reference" "R29"
-			(at 100.33 208.2801 0)
-			(show_name no)
-			(do_not_autoplace no)
-			(effects
-				(font
-					(size 1.27 1.27)
-				)
-				(justify left)
-			)
-		)
-		(property "Value" "2k2"
-			(at 100.33 205.7401 0)
-			(show_name no)
-			(do_not_autoplace no)
-			(effects
-				(font
-					(size 1.27 1.27)
-				)
-				(justify left)
-			)
-		)
-		(property "Footprint" "Resistor_SMD:R_0805_2012Metric"
-			(at 104.648 207.01 90)
-			(hide yes)
-			(show_name no)
-			(do_not_autoplace no)
-			(effects
-				(font
-					(size 1.27 1.27)
-				)
-			)
-		)
-		(property "Datasheet" ""
-			(at 102.87 207.01 0)
-			(hide yes)
-			(show_name no)
-			(do_not_autoplace no)
-			(effects
-				(font
-					(size 1.27 1.27)
-				)
-			)
-		)
-		(property "Description" ""
-			(at 102.87 207.01 0)
-			(show_name no)
-			(do_not_autoplace no)
-			(effects
-				(font
-					(size 1.27 1.27)
-				)
-			)
-		)
-		(pin "1"
-		)
-		(pin "2"
-		)
-		(instances
-			(project "esp32_xiaozhi"
-				(path "/cae338e8-f342-43cb-b99a-a0486629133c/7256592f-47bf-4ef9-8c00-e0996fdaf86a"
-					(reference "R29")
-					(unit 1)
-				)
-			)
-		)
-	)
-	(symbol
-		(lib_id "Device:R")
 		(at 234.95 118.11 0)
 		(unit 1)
@@
 					(unit 1)
 				)
+			)
+		)
+	)
+	(symbol
+		(lib_id "power:+5V")
+		(at 82.55 185.42 0)
+		(unit 1)
+		(body_style 1)
+		(exclude_from_sim no)
+		(in_bom yes)
+		(on_board yes)
+		(in_pos_files yes)
+		(dnp no)
+		(fields_autoplaced yes)
+		(property "Reference" "#PWR0142"
+			(at 82.55 189.23 0)
+			(hide yes)
+			(show_name no)
+			(do_not_autoplace no)
+			(effects
+				(font
+					(size 1.27 1.27)
+				)
+			)
+		)
+		(property "Value" "+5V"
+			(at 82.55 180.34 0)
+			(show_name no)
+			(do_not_autoplace no)
+			(effects
+				(font
+					(size 1.27 1.27)
+				)
+			)
+		)
+		(property "Footprint" ""
+			(at 82.55 185.42 0)
+			(hide yes)
+			(show_name no)
+			(do_not_autoplace no)
+			(effects
+				(font
+					(size 1.27 1.27)
+				)
+			)
+		)
+		(property "Datasheet" ""
+			(at 82.55 185.42 0)
+			(hide yes)
+			(show_name no)
+			(do_not_autoplace no)
+			(effects
+				(font
+					(size 1.27 1.27)
+				)
+			)
+		)
+		(property "Description" "Power symbol creates a global label with name \"+5V\""
+			(at 82.55 185.42 0)
+			(hide yes)
+			(show_name no)
+			(do_not_autoplace no)
+			(effects
+				(font
+					(size 1.27 1.27)
+				)
+			)
+		)
+		(pin "1"
+		)
+		(instances
+			(project "esp32_xiaozhi"
+				(path "/cae338e8-f342-43cb-b99a-a0486629133c/7256592f-47bf-4ef9-8c00-e0996fdaf86a"
+					(reference "#PWR0142")
+					(unit 1)
+				)

Commit message: Actualizaciones para versión single ESP32C6
Parts:
- removed D6: LED, Diode_SMD:D_0805_2012Metric, symbol Device:LED
- removed R30: 2k2, Resistor_SMD:R_0805_2012Metric, symbol Device:R
- added D15, D16: WS2812B, LED_SMD:LED_WS2812B_PLCC4_5.0x5.0mm_P3.2mm, symbol LED:WS2812B
Connections:
- net +5V: now also D15.1 (VDD), D16.1 (VDD)
- net GND: now also D15.3 (VSS), D16.3 (VSS)
- net at D7.2 (DOUT): now also D15.4 (DIN)
- new net: D15.2 (DOUT), D16.4 (DIN)
- no-connect marks 1 -> 0
Other:
- moved on the sheet: D13, D7, R39

Commit message: Update KiCad schematics/PCB and project files
Changed lines of the file:
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@@
 	)
 	(junction
-		(at 297.18 189.23)
+		(at 284.48 201.93)
 		(diameter 0)
 		(color 0 0 0 0)
@@
 	)
 	(junction
+		(at 307.34 201.93)
+		(diameter 0)
+		(color 0 0 0 0)
+	)
+	(junction
 		(at 273.05 143.51)
 		(diameter 0)
@@
 	)
 	(junction
+		(at 297.18 189.23)
+		(diameter 0)
+		(color 0 0 0 0)
+	)
+	(junction
 		(at 243.84 101.6)
 		(diameter 0)
@@
 	(wire
 		(pts
-			(xy 284.48 201.93) (xy 292.1 201.93)
+			(xy 276.86 201.93) (xy 284.48 201.93)
 		)
 		(stroke
@@
 	(wire
 		(pts
+			(xy 284.48 201.93) (xy 292.1 201.93)
+		)
+		(stroke
+			(width 0)
+			(type default)
+		)
+	)
+	(wire
+		(pts
 			(xy 234.95 143.51) (xy 251.46 143.51)
 		)
@@
 	(wire
 		(pts
+			(xy 297.18 186.69) (xy 297.18 189.23)
+		)
+		(stroke
+			(width 0)
+			(type default)
+		)
+	)
+	(wire
+		(pts
 			(xy 158.75 147.32) (xy 165.1 147.32)
 		)
@@
 	(wire
 		(pts
+			(xy 284.48 201.93) (xy 284.48 200.66)
+		)
+		(stroke
+			(width 0)
+			(type default)
+		)
+	)
+	(wire
+		(pts
 			(xy 125.73 147.32) (xy 137.16 147.32)
 		)
@@
 	(wire
 		(pts
-			(xy 186.69 123.19) (xy 186.69 121.92)
+			(xy 307.34 201.93) (xy 307.34 198.12)
 		)
 		(stroke
@@
 	(wire
 		(pts
-			(xy 148.59 237.49) (xy 148.59 240.03)
+			(xy 186.69 123.19) (xy 186.69 121.92)
 		)
 		(stroke
@@
 	(wire
 		(pts
-			(xy 92.71 195.58) (xy 92.71 185.42)
+			(xy 148.59 237.49) (xy 148.59 240.03)
 		)
 		(stroke
@@
 	(wire
 		(pts
-			(xy 243.84 101.6) (xy 234.95 101.6)
+			(xy 92.71 195.58) (xy 92.71 185.42)
 		)
 		(stroke
@@
 	(wire
 		(pts
-			(xy 284.48 200.66) (xy 284.48 201.93)
+			(xy 243.84 101.6) (xy 234.95 101.6)
 		)
 		(stroke
@@
 	(wire
 		(pts
-			(xy 176.53 106.68) (xy 186.69 106.68)
+			(xy 313.69 201.93) (xy 307.34 201.93)
 		)
 		(stroke
@@
 	(wire
 		(pts
-			(xy 243.84 130.81) (xy 251.46 130.81)
+			(xy 176.53 106.68) (xy 186.69 106.68)
 		)
 		(stroke
@@
 	(wire
 		(pts
-			(xy 158.75 134.62) (xy 165.1 134.62)
+			(xy 243.84 130.81) (xy 251.46 130.81)
 		)
 		(stroke
@@
 	(wire
 		(pts
-			(xy 187.96 121.92) (xy 187.96 119.38)
+			(xy 158.75 134.62) (xy 165.1 134.62)
 		)
 		(stroke
@@
 	(wire
 		(pts
-			(xy 307.34 201.93) (xy 307.34 198.12)
+			(xy 187.96 121.92) (xy 187.96 119.38)
 		)
 		(stroke
@@
 	(wire
 		(pts
-			(xy 307.34 189.23) (xy 307.34 190.5)
+			(xy 307.34 186.69) (xy 307.34 190.5)
 		)
 		(stroke
@@
 	(global_label "LED_Data_5V"
 		(shape input)
-		(at 307.34 199.39 0)
+		(at 313.69 201.93 0)
 		(fields_autoplaced yes)
 		(effects
@@
 		)
 		(property "Intersheetrefs" "${INTERSHEET_REFS}"
-			(at 322.2993 199.39 0)
+			(at 328.6493 201.93 0)
 			(hide yes)
 			(show_name no)
@@
 	(hierarchical_label "WS2812"
 		(shape input)
-		(at 284.48 201.93 180)
+		(at 276.86 201.93 180)
 		(effects
 			(font
@@
 	(symbol
 		(lib_id "power:+3V3")
-		(at 297.18 189.23 0)
+		(at 297.18 186.69 0)
 		(unit 1)
 		(body_style 1)
@@
 		(fields_autoplaced yes)
 		(property "Reference" "#PWR062"
-			(at 297.18 193.04 0)
+			(at 297.18 190.5 0)
 			(hide yes)
 			(show_name no)
@@
 		)
 		(property "Value" "+3V3"
-			(at 297.18 184.15 0)
+			(at 297.18 181.61 0)
 			(show_name no)
 			(do_not_autoplace no)
@@
 		)
 		(property "Footprint" ""
-			(at 297.18 189.23 0)
+			(at 297.18 186.69 0)
 			(hide yes)
 			(show_name no)
@@
 		)
 		(property "Datasheet" ""
-			(at 297.18 189.23 0)
+			(at 297.18 186.69 0)
 			(hide yes)
 			(show_name no)
@@
 		)
 		(property "Description" "Power symbol creates a global label with name \"+3V3\""
-			(at 297.18 189.23 0)
+			(at 297.18 186.69 0)
 			(hide yes)
 			(show_name no)
@@
 	(symbol
 		(lib_id "power:+5V")
-		(at 307.34 189.23 0)
+		(at 307.34 186.69 0)
 		(unit 1)
 		(body_style 1)
@@
 		(fields_autoplaced yes)
 		(property "Reference" "#PWR063"
-			(at 307.34 193.04 0)
+			(at 307.34 190.5 0)
 			(hide yes)
 			(show_name no)
@@
 		)
 		(property "Value" "+5V"
-			(at 309.88 187.9599 0)
+			(at 309.88 185.4199 0)
 			(show_name no)
 			(do_not_autoplace no)
@@
 		)
 		(property "Footprint" ""
-			(at 307.34 189.23 0)
+			(at 307.34 186.69 0)
 			(hide yes)
 			(show_name no)
@@
 		)
 		(property "Datasheet" ""
-			(at 307.34 189.23 0)
+			(at 307.34 186.69 0)
 			(hide yes)
 			(show_name no)
@@
 		)
 		(property "Description" ""
-			(at 307.34 189.23 0)
+			(at 307.34 186.69 0)
 			(show_name no)
 			(do_not_autoplace no)
