File: led_sw_gpio.kicad_sch (KiCad schematic)
At the start: 31 parts, among them Q6 2N7002, SW3 up, SW4 down, SW5 left, SW6 rigth, SW7 up, SW8 down

Commit message: add files update
Parts:
- D13: value LED -> WHITE
- D3: value LED -> BLUE
- D4: value LED -> GREEN
- R38: value 2k2 -> 10k
- R40: value 2k2 -> 10K
- SW7: value up -> Switch_push
- SW8: value down -> Switch_Push
Changed lines of the file:
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@@
 			)
 		)
-		(property "Description" ""
+		(property "Description" "Switch push  smd"
 			(at 151.13 147.32 0)
 			(show_name no)
@@
 		(in_pos_files yes)
 		(dnp no)
-		(fields_autoplaced yes)
 		(property "Reference" "D4"
 			(at 96.52 199.7074 90)
@@
 			)
 		)
-		(property "Value" "LED"
-			(at 96.52 202.2474 90)
+		(property "Value" "GREEN"
+			(at 96.52 189.992 0)
 			(show_name no)
 			(do_not_autoplace no)
@@
 			)
 		)
-		(property "Description" "Light emitting diode"
+		(property "Description" "Light emitting diode green"
 			(at 92.71 199.39 0)
 			(hide yes)
@@
 			)
 		)
-		(property "Description" ""
+		(property "Description" "Switch push  smd"
 			(at 201.93 123.19 0)
 			(show_name no)
@@
 			)
 		)
-		(property "Value" "LED"
+		(property "Value" "WHITE"
 			(at 109.22 202.2474 90)
 			(show_name no)
@@
 			)
 		)
-		(property "Description" "Light emitting diode"
+		(property "Description" "Light emitting diode white"
 			(at 105.41 199.39 0)
 			(hide yes)
@@
 		(in_pos_files yes)
 		(dnp no)
-		(fields_autoplaced yes)
 		(property "Reference" "#PWR0117"
 			(at 243.84 144.78 0)
@@
 		)
 		(property "Value" "GND"
-			(at 243.84 143.51 0)
+			(at 247.65 141.478 0)
 			(show_name no)
 			(do_not_autoplace no)
@@
 		(fields_autoplaced yes)
 		(property "Reference" "R38"
-			(at 281.94 198.1201 0)
+			(at 287.02 195.5799 0)
 			(show_name no)
 			(do_not_autoplace no)
@@
 					(size 1.27 1.27)
 				)
-				(justify left)
+				(justify right)
 			)
 		)
-		(property "Value" "2k2"
-			(at 281.94 195.5801 0)
+		(property "Value" "10k"
+			(at 287.02 198.1199 0)
 			(show_name no)
 			(do_not_autoplace no)
@@
 					(size 1.27 1.27)
 				)
-				(justify left)
+				(justify right)
 			)
 		)
@@
 		(in_pos_files yes)
 		(dnp no)
-		(fields_autoplaced yes)
 		(property "Reference" "D3"
 			(at 86.36 199.7074 90)
@@
 			)
 		)
-		(property "Value" "LED"
-			(at 86.36 202.2474 90)
+		(property "Value" "BLUE"
+			(at 70.612 195.072 90)
 			(show_name no)
 			(do_not_autoplace no)
@@
 			)
 		)
-		(property "Description" "Light emitting diode"
+		(property "Description" "Light emitting diode blue"
 			(at 82.55 199.39 0)
 			(hide yes)
@@
 			)
 		)
-		(property "Description" ""
+		(property "Description" "Switch push  smd"
 			(at 151.13 134.62 0)
 			(show_name no)
@@
 			)
 		)
-		(property "Value" "up"
+		(property "Value" "Switch_push"
 			(at 259.08 125.73 0)
 			(show_name no)
@@
 			)
 		)
-		(property "Description" ""
+		(property "Description" "Switch push  smd"
 			(at 259.08 130.81 0)
 			(show_name no)
@@
 		)
 		(property "Value" "WS2812B"
-			(at 153.67 241.3 0)
+			(at 137.16 239.268 0)
 			(show_name no)
 			(do_not_autoplace no)
@@
 		)
 		(property "Value" "WS2812B"
-			(at 184.15 241.3 0)
+			(at 179.832 231.648 0)
 			(show_name no)
 			(do_not_autoplace no)
@@
 			)
 		)
-		(property "Value" "down"
+		(property "Value" "Switch_Push"
 			(at 259.08 138.43 0)
 			(show_name no)
@@
 			)
 		)
-		(property "Description" ""
+		(property "Description" "Switch push  smd"
 			(at 259.08 143.51 0)
 			(show_name no)
@@
 		)
 		(property "Value" "WS2812B"
-			(at 168.91 241.3 0)
+			(at 162.052 233.934 0)
 			(show_name no)
 			(do_not_autoplace no)
@@
 			)
 		)
-		(property "Description" ""
+		(property "Description" "Switch push  smd"
 			(at 201.93 135.89 0)
 			(show_name no)
@@
 		(fields_autoplaced yes)
 		(property "Reference" "R40"
-			(at 304.8 195.5801 0)
+			(at 309.88 193.0399 0)
 			(show_name no)
 			(do_not_autoplace no)
@@
 					(size 1.27 1.27)
 				)
-				(justify left)
+				(justify right)
 			)
 		)
-		(property "Value" "2k2"
-			(at 304.8 193.0401 0)
+		(property "Value" "10K"
+			(at 309.88 195.5799 0)
 			(show_name no)
 			(do_not_autoplace no)
@@
 					(size 1.27 1.27)
 				)
-				(justify left)
+				(justify right)
 			)
 		)
