File: epaper.kicad_sch (KiCad schematic)
At the start: 36 parts, among them J25 TP_VCC, J26 IDC40, J53 F32R-1A7H1-11024, J54 tp_epaper, J56 tp_epaper, J57 tp_epaper, J58 tp_epaper, J59 tp_epaper, Q1 PMOS, Q12 FDN306P, Q13 FDN306P, Q15 2N7002

Commit message: actualizacion  de pcb logic , rpi
Parts:
- J53: Package None -> (none)
- Q12, Q13: Package TO-236-3 ON -> (none)
Changed lines of the file:
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@@
 			)
 		)
-		(property "Package" "None"
-			(at 339.09 119.38 0)
-			(hide yes)
-			(show_name no)
-			(do_not_autoplace no)
-			(effects
-				(font
-					(size 1.27 1.27)
-				)
-				(justify bottom)
-			)
-		)
 		(property "Price" "None"
 			(at 339.09 119.38 0)
@@
 			)
 		)
-		(property "Package" "TO-236-3 ON"
-			(at 190.5 190.5 0)
-			(hide yes)
-			(show_name no)
-			(do_not_autoplace no)
-			(effects
-				(font
-					(size 1.27 1.27)
-				)
-				(justify bottom)
-			)
-		)
 		(property "Price" "None"
 			(at 190.5 190.5 0)
@@
 			(at 166.37 196.85 0)
 			(hide yes)
-			(show_name no)
-			(do_not_autoplace no)
-			(effects
-				(font
-					(size 1.27 1.27)
-				)
-				(justify bottom)
-			)
-		)
-		(property "Package" "TO-236-3 ON"
-			(at 166.37 196.85 0)
-			(hide yes)
