File: logic_dip28.kicad_sch (KiCad schematic)
At the start: 19 parts, among them J34 Raspberry_Pi_zero_2w, Q2 BC846, Q3 2N7002, Q8 2N7002, U16 TXS0108, U17 TXS0108, U18 TXS0108, U19 M48T08-150PC

Commit message: actualizacion  de pcb logic , rpi
Parts:
- C82, C83, C84, C85, C86, Q3, Q8: now left out of the parts list
- U19: Package DIP-28 STMicroelectronics -> (none)
Changed lines of the file:
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@@
 		(body_style 1)
 		(exclude_from_sim no)
-		(in_bom yes)
+		(in_bom no)
 		(on_board yes)
-		(in_pos_files yes)
+		(in_pos_files no)
 		(dnp no)
 		(fields_autoplaced yes)
@@
 		(body_style 1)
 		(exclude_from_sim no)
-		(in_bom yes)
+		(in_bom no)
 		(on_board yes)
-		(in_pos_files yes)
+		(in_pos_files no)
 		(dnp no)
 		(fields_autoplaced yes)
@@
 		(body_style 1)
 		(exclude_from_sim no)
-		(in_bom yes)
+		(in_bom no)
 		(on_board yes)
-		(in_pos_files yes)
+		(in_pos_files no)
 		(dnp no)
 		(property "Reference" "C84"
@@
 			)
 		)
-		(property "Package" "DIP-28 STMicroelectronics"
-			(at 311.15 135.89 0)
-			(hide yes)
-			(show_name no)
-			(do_not_autoplace no)
-			(effects
-				(font
-					(size 1.27 1.27)
-				)
-				(justify bottom)
-			)
-		)
 		(property "OC_FARNELL" "9756540"
 			(at 311.15 135.89 0)
@@
 		(body_style 1)
 		(exclude_from_sim no)
-		(in_bom yes)
+		(in_bom no)
 		(on_board yes)
-		(in_pos_files yes)
+		(in_pos_files no)
 		(dnp no)
 		(property "Reference" "C82"
@@
 		(body_style 1)
 		(exclude_from_sim no)
-		(in_bom yes)
+		(in_bom no)
 		(on_board yes)
-		(in_pos_files yes)
+		(in_pos_files no)
 		(dnp no)
 		(property "Reference" "C83"
@@
 		(body_style 1)
 		(exclude_from_sim no)
-		(in_bom yes)
+		(in_bom no)
 		(on_board yes)
-		(in_pos_files yes)
+		(in_pos_files no)
 		(dnp no)
 		(property "Reference" "C85"
@@
 		(body_style 1)
 		(exclude_from_sim no)
-		(in_bom yes)
+		(in_bom no)
 		(on_board yes)
-		(in_pos_files yes)
+		(in_pos_files no)
 		(dnp no)
 		(property "Reference" "C86"

Commit message: add update
Parts:
- added J27: oled, Connector_PinHeader_2.54mm:PinHeader_1x04_P2.54mm_Vertical, symbol Connector:Conn_01x04_Pin
- U19: now not fitted
Connections:
- net +3V3C: now also J27.2 (Pin_2)
- net GND: now also J27.1 (Pin_1)
- net GPIO2: now also J27.4 (Pin_4)
- net GPIO3: now also J27.3 (Pin_3)
